File: Draco.kicad_pcb (KiCad board)
At the start: 2 copper layers, 106 parts, among them J1 Conn_01x03, J10 Conn_01x03, J11 Conn_01x06, J12 Conn_02x05_Odd_Even, J13 Conn_01x04, J14 Conn_01x01, J15 Micro_SD_Card, J16 Conn_01x03, J17 CHARGE_A, J18 CHARGE_C, J19 CHARGE_B, J2 Conn_01x03, J3 Conn_01x03, J4 Conn_01x03, J5 Conn_01x03, J6 Conn_01x03, J7 Conn_01x03, J8 Conn_01x03, J9 Conn_01x03, Q1 BC817, Q2 Q_NMOS_DGS, Q3 BC817, Q4 Q_NMOS_DGS, Q5 BC817, Q6 Q_NMOS_DGS, U1 ATMEGA2560-16AU, U2 LOGIC-TXS0108EPWR(TSSOP20), U3 RFM95HW, U4 LM2574-5.0V, U5 LM2574-3.3V, U6 SAM-M8Q, U7 BMX055, U8 MS5607, Y1 16MHz

Commit message: Finished charge layout
Parts:
- added REF**: MountingHole_2.5mm_Pad_Via, Mounting_Holes:MountingHole_2.5mm_Pad_Via, F.Cu at (168.4, 79.7)
- moved C19 458.8 mm to (108.8, 35.9), turned to 180 degrees
- moved R29 455.8 mm to (62.6, 43.8), turned to 0 degrees
- moved J16 454.5 mm to (63.5, 51.4)
- moved R30 452.9 mm to (66.2, 44.1), turned to 0 degrees
- moved D6 445.0 mm to (126.7, 27.1), turned to 180 degrees
- moved JP2 432.6 mm to (88.6, 40.6)
- moved C21 431.8 mm to (159.1, 37.7), turned to 180 degrees
- moved C17 425.8 mm to (110.1, 31.1), turned to 90 degrees
- moved C20 423.3 mm to (161.9, 51.4), turned to 270 degrees
- moved L3 422.2 mm to (127.5, 31.4), turned to 270 degrees
- moved D4 418.0 mm to (111.9, 35.4), turned to 270 degrees
- moved U5 417.3 mm to (165.9, 40.5), turned to 270 degrees
- moved C16 415.9 mm to (105.4, 32.1), turned to 180 degrees
- moved C24 415.1 mm to (147.6, 46.2), turned to 90 degrees
- moved C15 414.2 mm to (106.3, 29.5), turned to 90 degrees
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Connections:
- U4 pad 1: +5V -> (no net)
- U4 pad 10: (no net) -> Net-(D4-Pad1)
- U4 pad 12: (no net) -> Net-(D6-Pad1)
- U4 pad 2: GND -> (no net)
- U4 pad 3: GND -> +5V
- U4 pad 5: Net-(D4-Pad1) -> GND
- U4 pad 6: (no net) -> GND
- U4 pad 7: Net-(D6-Pad1) -> (no net)
- U5 pad 1: +3V3 -> (no net)
- U5 pad 10: (no net) -> +5V
- U5 pad 12: (no net) -> Net-(D5-Pad1)
- U5 pad 2: GND -> (no net)
- U5 pad 3: GND -> +3V3
- U5 pad 5: +5V -> GND
- U5 pad 6: (no net) -> GND
- U5 pad 7: Net-(D5-Pad1) -> (no net)
Routing:
- net GND: track 0.00 -> 163.2 mm
- net Net-(J18-Pad2): track 0.00 -> 55.7 mm, vias 0 -> 1
- net +BATT: track 0.00 -> 47.5 mm
- net Net-(J1-Pad2): track 0.00 -> 38.9 mm
- net Net-(BT1-Pad1): track 0.00 -> 35.3 mm
- net Net-(J17-Pad2): track 0.00 -> 33.0 mm, vias 0 -> 1
- net +3V3: track 0.00 -> 32.0 mm
- net Net-(J19-Pad2): track 0.00 -> 26.9 mm, vias 0 -> 1
- net Net-(D6-Pad1): track 0.00 -> 21.9 mm
- net Net-(Q6-Pad2): track 0.00 -> 12.6 mm
- net +5V: track 0.00 -> 10.6 mm
- net Net-(Q2-Pad2): track 0.00 -> 9.26 mm
- net Net-(Q4-Pad2): track 0.00 -> 9.08 mm
- net Net-(AE1-Pad1): track 0.00 -> 7.56 mm
- net Net-(D4-Pad1): track 0.00 -> 7.27 mm
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Other:
- board outline added: 95.2 x 44.5 mm

Commit message: Started board placement
Parts:
- removed the REF** at (168.4, 79.7)
- added REF**: MountingHole_2.5mm_Pad_Via, Mounting_Holes:MountingHole_2.5mm_Pad_Via, F.Cu at (168.5, 117.7)
- added REF**: MountingHole_2.5mm_Pad_Via, Mounting_Holes:MountingHole_2.5mm_Pad_Via, F.Cu at (168.5, 79.1)
- moved U1 347.3 mm to (127.0, 99.8)
- moved JP1 254.4 mm to (103.8, 118.6)
- moved J1 210.8 mm to (108.7, 113.7)
- moved J10 210.8 mm to (143.0, 113.7)
- moved J2 210.8 mm to (112.5, 113.7)
- moved J3 210.8 mm to (116.3, 113.7)
- moved J4 210.8 mm to (120.1, 113.7)
- moved J5 210.8 mm to (124.0, 113.7)
- moved J6 210.8 mm to (127.8, 113.7)
- moved J7 210.8 mm to (131.6, 113.7)
- moved J8 210.8 mm to (135.4, 113.7)
- moved J9 210.8 mm to (139.2, 113.7)
- moved Q2 37.0 mm to (156.2, 92.8)
- moved Q4 37.0 mm to (156.2, 85.7)
- moved Q6 37.0 mm to (156.2, 99.9)
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Routing:
- net /~FIRE_C: track 1.92 -> 23.2 mm, vias 0 -> 2
- net /~FIRE_A: track 1.90 -> 19.9 mm
- net /~FIRE_B: track 1.90 -> 18.1 mm
- net /SERVO6: track 0.00 -> 6.24 mm
- net Net-(J1-Pad2): track 38.9 -> 34.3 mm

Commit message: Routed crystal; might not be permenant spot
Parts:
- moved C5 304.5 mm to (123.7, 107.5)
- moved Y1 304.5 mm to (115.9, 108.4)
- moved C4 304.4 mm to (108.2, 109.2), turned to 270 degrees
- moved U1 2.84 mm to (127.0, 97.0)
- moved JP1 1.40 mm to (102.4, 118.6)
Routing:
- net /SERVO1: track 0.00 -> 24.1 mm
- net /~FIRE_C: track 23.2 -> 2.12 mm, vias 2 -> 0
- net /SERVO2: track 0.00 -> 21.0 mm
- net Net-(C4-Pad1): track 0.00 -> 19.7 mm
- net GND: track 163.2 -> 182.7 mm
- net /SERVO3: track 0.00 -> 18.0 mm
- net /~FIRE_A: track 19.9 -> 2.02 mm
- net /~FIRE_B: track 18.1 -> 1.90 mm
- net /SERVO4: track 0.00 -> 15.0 mm
- net /SERVO5: track 0.00 -> 12.0 mm
- net Net-(C5-Pad1): track 0.00 -> 8.38 mm
- net /SERVO6: track 6.24 -> 9.09 mm
- net /SERVO7: track 0.00 -> 0.63 mm

Commit message: pushed new psu to pcb
Parts:
- removed D6: 11DQ06, Diodes_THT:D_DO-41_SOD81_P2.54mm_Vertical_AnodeUp
- removed REF** (x2): MountingHole_2.5mm_Pad_Via, Mounting_Holes:MountingHole_2.5mm_Pad_Via
- added C30, C31: 10uF, Capacitors_SMD:C_0805, F.Cu at (123.8, 130.7)
- added R31, R34: 10k2, Resistors_SMD:R_0805, F.Cu at (123.8, 130.7)
- added R32: 453k, Resistors_SMD:R_0805, F.Cu at (123.8, 130.7)
- added R33: 97.6k, Resistors_SMD:R_0805, F.Cu at (123.8, 130.7)
- added R35: 1k96, Resistors_SMD:R_0805, F.Cu at (123.8, 130.7)
- C11, C17, C9: footprint Capacitors_THT:CP_Radial_D5.0mm_P2.00mm -> Capacitors_SMD:C_0805
- C16, C23: value 100nF -> 22uF
- C18: value 100nF -> 120pF 50V
- C19: value 22uF -> 4.7uF; footprint Capacitors_THT:CP_Radial_D5.0mm_P2.00mm -> Capacitors_SMD:C_0805
- C20: value 100nF -> 6.8nF 50V
- C21: value 200uF -> 8.2nF; footprint Capacitors_THT:CP_Radial_D5.0mm_P2.00mm -> Capacitors_SMD:C_0805
- C22: value 200uF -> 100nF; footprint Capacitors_THT:CP_Radial_D5.0mm_P2.00mm -> Capacitors_SMD:C_0805
- C24: value 100nF -> 10uF
- D4: value B0520LW-7-F -> 30V 1.5A 400mV Vf; footprint Diodes_SMD:D_SOD-123 -> Diodes_SMD:D_SOD-323
- D5: value 11DQ06 -> 0.55V 1A; footprint Diodes_THT:D_DO-41_SOD81_P2.54mm_Vertical_AnodeUp -> Diodes_SMD:D_SOD-123F
- L2: value 100uH 0.5A -> 2.2uH; footprint Inductors_THT:L_Radial_D8.7mm_P5.00mm_Fastron_07HCP -> Inductors_SMD:L_Taiyo-Yuden_NR-60xx
- L3: value 330uF 1A -> 15uH 0.096ohm; footprint Inductors_THT:L_Radial_D8.7mm_P5.00mm_Fastron_07HCP -> Inductors_SMD:L_Taiyo-Yuden_NR-60xx
- R29, R30: value 10K -> 47K
- U4: value LM2574-5.0V -> TPS54332; footprint Housings_SOIC:SOIC-14W_7.5x9.0mm_Pitch1.27mm -> Housings_SOIC:SOIC-8-1EP_3.9x4.9mm_Pitch1.27mm
- U5: value LM2574-3.3V -> TLV62568; footprint Housings_SOIC:SOIC-14W_7.5x9.0mm_Pitch1.27mm -> TO_SOT_Packages_SMD:SOT-23-5
- moved U2 57.9 mm to (435.4, 80.7)
- moved Y1 50.5 mm to (93.2, 153.4)
- moved C4 41.4 mm to (103.4, 150.4)
- moved C5 40.5 mm to (111.0, 145.9)
- moved C23 19.0 mm to (164.6, 45.3), turned to 0 degrees
- moved L2 15.3 mm to (160.3, 40.3)
- moved D4 11.1 mm to (118.3, 26.3), turned to 90 degrees
- moved C19 11.0 mm to (119.8, 36.7)
- moved C22 9.88 mm to (150.6, 38.4)
- moved C21 6.70 mm to (153.6, 34.0)
- moved L3 3.83 mm to (123.7, 31.8), turned to 90 degrees
- moved C15 3.26 mm to (109.1, 31.2), turned to 270 degrees
- moved C16 2.06 mm to (107.2, 31.2), turned to 270 degrees
- moved JP1 1.43 mm to (103.8, 118.7)
- moved U4 1.22 mm to (117.6, 31.7)
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Connections:
- C18 pad 1: +3V3 -> Net-(C18-Pad1)
- C19 pad 1: +BATT -> +5V
- C20 pad 1: +3V3 -> Net-(C20-Pad1)
- C21 pad 1: +3V3 -> Net-(C21-Pad1)
- C22 pad 1: +5V -> Net-(C22-Pad1)
- C22 pad 2: GND -> Net-(C22-Pad2)
- C23 pad 1: +5V -> +3V3
- D5 pad 1: Net-(D5-Pad1) -> Net-(C22-Pad2)
- L2 pad 1: +3V3 -> Net-(L2-Pad1)
- L2 pad 2: Net-(D5-Pad1) -> +3V3
- L3 pad 1: +5V -> Net-(C22-Pad2)
- L3 pad 2: Net-(D6-Pad1) -> +5V
- U4 pad 1: (no net) -> Net-(C22-Pad1)
- U4 pad 2: (no net) -> Net-(D4-Pad1)
- U4 pad 3: +5V -> Net-(U4-Pad3)
- U4 pad 4: GND -> Net-(C21-Pad1)
- U4 pad 5: GND -> Net-(R34-Pad2)
- U4 pad 6: GND -> Net-(C18-Pad1)
- U4 pad 7: (no net) -> GND
- U4 pad 8: (no net) -> Net-(C22-Pad2)
- U4 pad 9: (no net) -> GND
- U5 pad 1: (no net) -> +5V
- U5 pad 2: (no net) -> GND
- U5 pad 3: +3V3 -> Net-(L2-Pad1)
- U5 pad 4: GND -> +5V
- U5 pad 5: GND -> Net-(R32-Pad2)
Routing:
- net GND: track 182.7 -> 131.0 mm
- net Net-(D6-Pad1): track 21.9 -> 0.00 mm
- net Net-(C4-Pad1): track 19.7 -> 0.00 mm
- net +BATT: track 47.5 -> 33.1 mm
- net /SERVO8: track 0.00 -> 14.2 mm
- net /SERVO7: track 0.63 -> 11.6 mm
- net +5V: track 10.6 -> 0.00 mm
- net Net-(C5-Pad1): track 8.38 -> 0.00 mm
- net Net-(D4-Pad1): track 7.27 -> 1.65 mm
- net Net-(C22-Pad2): track 0.00 -> 4.31 mm

Commit message: Doing PCB Layout
Parts:
- moved C18 65.5 mm to (133.1, 47.0)
- moved D5 52.6 mm to (122.7, 41.9)
- moved C21 39.9 mm to (113.9, 29.7), turned to 270 degrees
- moved C22 30.1 mm to (122.7, 27.0), turned to 0 degrees
- moved C24 21.9 mm to (129.7, 33.7), turned to 270 degrees
- moved C19 8.63 mm to (127.9, 33.7), turned to 270 degrees
- moved C20 6.10 mm to (158.8, 46.2)
- moved L3 0.25 mm to (123.7, 32.0)
Routing:
- net GND: track 131.0 -> 146.6 mm
- net +5V: track 0.00 -> 6.51 mm
- net Net-(C21-Pad1): track 0.00 -> 1.88 mm
Changed lines of the file:
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@@
   (general
     (links 304)
-    (no_connects 200)
-    (area 76.124999 76.124999 171.525001 120.725001)
+    (no_connects 196)
+    (area 52.225 -32.731 560.247001 158.041)
     (thickness 1.6)
     (drawings 6)
-    (tracks 269)
+    (tracks 281)
     (zones 0)
     (modules 112)
@@
   )
   (setup
-    (last_trace_width 0.25)
+    (last_trace_width 1)
     (user_trace_width 1)
     (user_trace_width 2)
@@
   )
   (module Capacitors_SMD:C_0805 (layer F.Cu)
-    (at 198.12 54.991)
+    (at 133.096 46.99)
     (descr "Capacitor SMD 0805, reflow soldering, AVX (see smccp.pdf)")
     (tags "capacitor 0805")
@@
   )
   (module Capacitors_SMD:C_0805 (layer F.Cu)
-    (at 161.925 51.435 270)
+    (at 158.75 46.228 270)
     (descr "Capacitor SMD 0805, reflow soldering, AVX (see smccp.pdf)")
     (tags "capacitor 0805")
@@
   )
   (module Capacitors_SMD:C_0805 (layer F.Cu)
-    (at 147.574 46.228 90)
+    (at 129.667 33.7058 270)
     (descr "Capacitor SMD 0805, reflow soldering, AVX (see smccp.pdf)")
     (tags "capacitor 0805")
     (attr smd)
-    (fp_text reference C24 (at 0 -1.5 90) (layer F.SilkS)
+    (fp_text reference C24 (at 0 -1.5 270) (layer F.SilkS)
       (effects (font (size 1 1) (thickness 0.15)))
     )
-    (fp_text value 10uF (at 0 1.75 90) (layer F.Fab)
+    (fp_text value 10uF (at 0 1.75 270) (layer F.Fab)
       (effects (font (size 1 1) (thickness 0.15)))
     )
-    (fp_text user %R (at 0 -1.5 90) (layer F.Fab)
+    (fp_text user %R (at 0 -1.5 270) (layer F.Fab)
       (effects (font (size 1 1) (thickness 0.15)))
     )
@@
     (fp_line (start 1.75 0.87) (end 1.75 -0.88) (layer F.CrtYd) (width 0.05))
     (fp_line (start 1.75 0.87) (end -1.75 0.87) (layer F.CrtYd) (width 0.05))
-    (pad 1 smd rect (at -1 0 90) (size 1 1.25) (layers F.Cu F.Paste F.Mask)
+    (pad 1 smd rect (at -1 0 270) (size 1 1.25) (layers F.Cu F.Paste F.Mask)
       (net 4 +5V))
-    (pad 2 smd rect (at 1 0 90) (size 1 1.25) (layers F.Cu F.Paste F.Mask)
+    (pad 2 smd rect (at 1 0 270) (size 1 1.25) (layers F.Cu F.Paste F.Mask)
       (net 1 GND))
     (model Capacitors_SMD.3dshapes/C_0805.wrl
@@
   )
   (module Capacitors_SMD:C_0805 (layer F.Cu)
-    (at 119.7864 36.6776 180)
+    (at 127.889 33.7185 270)
     (descr "Capacitor SMD 0805, reflow soldering, AVX (see smccp.pdf)")
     (tags "capacitor 0805")
     (attr smd)
-    (fp_text reference C19 (at 0 -1.5 180) (layer F.SilkS)
+    (fp_text reference C19 (at 0 -1.5 270) (layer F.SilkS)
       (effects (font (size 1 1) (thickness 0.15)))
     )
-    (fp_text value 4.7uF (at 0 1.75 180) (layer F.Fab)
+    (fp_text value 4.7uF (at 0 1.75 270) (layer F.Fab)
       (effects (font (size 1 1) (thickness 0.15)))
     )
-    (fp_text user %R (at 0 -1.5 180) (layer F.Fab)
+    (fp_text user %R (at 0 -1.5 270) (layer F.Fab)
       (effects (font (size 1 1) (thickness 0.15)))
     )
@@
     (fp_line (start 1.75 0.87) (end 1.75 -0.88) (layer F.CrtYd) (width 0.05))
     (fp_line (start 1.75 0.87) (end -1.75 0.87) (layer F.CrtYd) (width 0.05))
-    (pad 1 smd rect (at -1 0 180) (size 1 1.25) (layers F.Cu F.Paste F.Mask)
+    (pad 1 smd rect (at -1 0 270) (size 1 1.25) (layers F.Cu F.Paste F.Mask)
       (net 4 +5V))
-    (pad 2 smd rect (at 1 0 180) (size 1 1.25) (layers F.Cu F.Paste F.Mask)
+    (pad 2 smd rect (at 1 0 270) (size 1 1.25) (layers F.Cu F.Paste F.Mask)
       (net 1 GND))
     (model Capacitors_SMD.3dshapes/C_0805.wrl
@@
   )
   (module Capacitors_SMD:C_0805 (layer F.Cu)
-    (at 153.5684 33.9852 180)
+    (at 113.9444 29.6926 270)
     (descr "Capacitor SMD 0805, reflow soldering, AVX (see smccp.pdf)")
     (tags "capacitor 0805")
     (attr smd)
-    (fp_text reference C21 (at 0 -1.5 180) (layer F.SilkS)
+    (fp_text reference C21 (at 0 -1.5 270) (layer F.SilkS)
       (effects (font (size 1 1) (thickness 0.15)))
     )
-    (fp_text value 8.2nF (at 0 1.75 180) (layer F.Fab)
+    (fp_text value 8.2nF (at 0 1.75 270) (layer F.Fab)
       (effects (font (size 1 1) (thickness 0.15)))
     )
-    (fp_text user %R (at 0 -1.5 180) (layer F.Fab)
+    (fp_text user %R (at 0 -1.5 270) (layer F.Fab)
       (effects (font (size 1 1) (thickness 0.15)))
     )
@@
     (fp_line (start 1.75 0.87) (end 1.75 -0.88) (layer F.CrtYd) (width 0.05))
     (fp_line (start 1.75 0.87) (end -1.75 0.87) (layer F.CrtYd) (width 0.05))
-    (pad 1 smd rect (at -1 0 180) (size 1 1.25) (layers F.Cu F.Paste F.Mask)
+    (pad 1 smd rect (at -1 0 270) (size 1 1.25) (layers F.Cu F.Paste F.Mask)
       (net 152 "Net-(C21-Pad1)"))
-    (pad 2 smd rect (at 1 0 180) (size 1 1.25) (layers F.Cu F.Paste F.Mask)
+    (pad 2 smd rect (at 1 0 270) (size 1 1.25) (layers F.Cu F.Paste F.Mask)
       (net 1 GND))
     (model Capacitors_SMD.3dshapes/C_0805.wrl
@@
   )
   (module Capacitors_SMD:C_0805 (layer F.Cu)
-    (at 150.622 38.4048 180)
+    (at 122.7328 26.9748)
     (descr "Capacitor SMD 0805, reflow soldering, AVX (see smccp.pdf)")
     (tags "capacitor 0805")
     (attr smd)
-    (fp_text reference C22 (at 0 -1.5 180) (layer F.SilkS)
+    (fp_text reference C22 (at 0 -1.5) (layer F.SilkS)
       (effects (font (size 1 1) (thickness 0.15)))
     )
-    (fp_text value 100nF (at 0 1.75 180) (layer F.Fab)
+    (fp_text value 100nF (at 0 1.75) (layer F.Fab)
       (effects (font (size 1 1) (thickness 0.15)))
     )
-    (fp_text user %R (at 0 -1.5 180) (layer F.Fab)
+    (fp_text user %R (at 0 -1.5) (layer F.Fab)
       (effects (font (size 1 1) (thickness 0.15)))
     )
@@
     (fp_line (start 1.75 0.87) (end 1.75 -0.88) (layer F.CrtYd) (width 0.05))
     (fp_line (start 1.75 0.87) (end -1.75 0.87) (layer F.CrtYd) (width 0.05))
-    (pad 1 smd rect (at -1 0 180) (size 1 1.25) (layers F.Cu F.Paste F.Mask)
+    (pad 1 smd rect (at -1 0) (size 1 1.25) (layers F.Cu F.Paste F.Mask)
       (net 153 "Net-(C22-Pad1)"))
-    (pad 2 smd rect (at 1 0 180) (size 1 1.25) (layers F.Cu F.Paste F.Mask)
+    (pad 2 smd rect (at 1 0) (size 1 1.25) (layers F.Cu F.Paste F.Mask)
       (net 154 "Net-(C22-Pad2)"))
     (model Capacitors_SMD.3dshapes/C_0805.wrl
@@
   )
   (module Diodes_SMD:D_SOD-123F (layer F.Cu)
-    (at 174.752 34.671 180)
+    (at 122.682 41.91 180)
     (descr D_SOD-123F)
     (tags D_SOD-123F)
@@
   )
   (module Inductors_SMD:L_Taiyo-Yuden_NR-60xx (layer F.Cu)
-    (at 123.698 31.75 90)
+    (at 123.698 32.004 90)
     (descr "Inductor, Taiyo Yuden, NR series, Taiyo-Yuden_NR-60xx, 6.0mmx6.0mm")
     (tags "inductor taiyo-yuden nr smd")
@@
   (segment (start 156.3878 106.3498) (end 156.5402 106.3498) (width 0.25) (layer B.Cu) (net 0))
   (segment (start 106.299 32.02) (end 106.41 32.131) (width 1) (layer F.Cu) (net 0))
+  (segment (start 113.9444 30.6926) (end 116.5954 30.6926) (width 1) (layer F.Cu) (net 1))
+  (segment (start 116.5954 30.6926) (end 117.0145 31.1117) (width 1) (layer F.Cu) (net 1))
+  (segment (start 118.237 34.3992) (end 118.237 35.6235) (width 1) (layer F.Cu) (net 1))
+  (segment (start 127.889 35.8775) (end 127.889 34.7185) (width 1) (layer F.Cu) (net 1))
+  (segment (start 127.5715 36.195) (end 127.889 35.8775) (width 1) (layer F.Cu) (net 1))
+  (segment (start 118.8085 36.195) (end 127.5715 36.195) (width 1) (layer F.Cu) (net 1))
+  (segment (start 118.237 35.6235) (end 118.8085 36.195) (width 1) (layer F.Cu) (net 1))
   (segment (start 118.1895 32.2867) (end 118.1895 34.3517) (width 1) (layer F.Cu) (net 1))
   (segment (start 118.1895 34.3517) (end 118.237 34.3992) (width 1) (layer F.Cu) (net 1))
@@
   (segment (start 419.1 129.286) (end 419.1 119.862) (width 1) (layer F.Cu) (net 3))
   (segment (start 419.1 119.862) (end 423.037 115.925) (width 1) (layer F.Cu) (net 3))
+  (segment (start 127.889 32.7185) (end 127.889 30.9245) (width 1) (layer F.Cu) (net 4))
+  (segment (start 127.889 30.9245) (end 126.6185 29.654) (width 1) (layer F.Cu) (net 4))
+  (segment (start 126.6185 29.654) (end 123.698 29.654) (width 1) (layer F.Cu) (net 4))
   (segment (start 498.348 89.8365) (end 499.1295 89.8365) (width 0.25) (layer F.Cu) (net 10))
   (segment (start 499.1295 89.8365) (end 500.126 88.84) (width 0.25) (layer F.Cu) (net 10))
@@
   (segment (start 502.326 86.34) (end 506.049 86.34) (width 0.25) (layer F.Cu) (net 78))
   (segment (start 506.049 86.34) (end 506.095 86.294) (width 0.25) (layer F.Cu) (net 78))
-  (segment (start 119.507 34.3992) (end 123.3988 34.3992) (width 1) (layer F.Cu) (net 154))
-  (segment (start 123.3988 34.3992) (end 123.698 34.1) (width 1) (layer F.Cu) (net 154))
+  (segment (start 115.697 28.9992) (end 114.251 28.9992) (width 1) (layer F.Cu) (net 152))
+  (segment (start 114.251 28.9992) (end 113.9444 28.6926) (width 1) (layer F.Cu) (net 152))
+  (segment (start 119.507 34.3992) (end 123.3988 34.6532) (width 1) (layer F.Cu) (net 154) (status 20))
+  (segment (start 123.3988 34.6532) (end 123.698 34.354) (width 1) (layer F.Cu) (net 154) (status 30))
 )

Commit message: moved charge module, routed lots of stuff
Parts:
- added J20: Conn_01x04, Pin_Headers:Pin_Header_Angled_1x04_Pitch2.54mm, F.Cu at (123.8, 130.7)
- added REF**: MountingHole_2.2mm_M2_Pad, Mounting_Holes:MountingHole_2.2mm_M2_Pad, F.Cu at (168.8, 78.9)
- added REF**: MountingHole_2.2mm_M2_Pad, Mounting_Holes:MountingHole_2.2mm_M2_Pad, F.Cu at (168.8, 118.0)
- added REF**: MountingHole_2.2mm_M2_Pad, Mounting_Holes:MountingHole_2.2mm_M2_Pad, F.Cu at (78.9, 118.0)
- added REF**: MountingHole_2.2mm_M2_Pad, Mounting_Holes:MountingHole_2.2mm_M2_Pad, F.Cu at (78.9, 78.9)
- moved R33 99.0 mm to (152.3, 35.9), turned to 180 degrees
- moved R32 98.4 mm to (156.0, 37.7), turned to 90 degrees
- moved C20 94.3 mm to (97.4, 117.9), turned to 180 degrees
- moved D4 93.2 mm to (90.7, 115.3), turned to 270 degrees
- moved C17 89.8 mm to (90.7, 118.7)
- moved C15 89.0 mm to (92.6, 118.7)
- moved C21 88.8 mm to (93.4, 116.1), turned to 0 degrees
- moved C16 88.5 mm to (94.5, 118.7)
- moved C24 87.8 mm to (106.7, 118.4)
- moved C22 86.2 mm to (95.3, 108.7)
- moved U4 83.7 mm to (95.4, 112.4), turned to 0 degrees
- moved L3 80.2 mm to (105.0, 110.0), turned to 0 degrees
- moved C18 77.7 mm to (97.4, 116.1), turned to 180 degrees
- moved J18 76.7 mm to (89.9, 81.5), turned to 180 degrees
- moved Q4 74.6 mm to (81.7, 91.1), turned to 270 degrees
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Connections:
- J17 pad 1: +BATT -> VCC
- J18 pad 1: +BATT -> VCC
- J19 pad 1: +BATT -> VCC
- JP1 pad 1: VCC -> +BATT
Routing:
- net VCC: track 0.00 -> 81.4 mm
- net GND: track 146.6 -> 216.6 mm
- net Net-(J18-Pad2): track 55.7 -> 5.71 mm, vias 1 -> 0
- net Net-(J17-Pad2): track 33.0 -> 9.80 mm, vias 1 -> 0
- net /SERVO1: track 24.1 -> 0.91 mm
- net /SERVO2: track 21.0 -> 0.03 mm
- net +5V: track 6.51 -> 26.1 mm
- net Net-(J1-Pad2): track 34.3 -> 52.9 mm
- net /SERVO3: track 18.0 -> 0.13 mm
- net /SERVO4: track 15.0 -> 0.13 mm
- net Net-(J19-Pad2): track 26.9 -> 12.3 mm, vias 1 -> 0
- net /SERVO8: track 14.2 -> 0.00 mm
- net /SERVO5: track 12.0 -> 0.33 mm
- net /SERVO7: track 11.6 -> 0.64 mm
- net Net-(C18-Pad1): track 0.00 -> 10.6 mm
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
Commit message: moving blocks around
Parts:
- BT1, C25, C26, R2, R3, U6: moved to B.Cu
- moved R3 247.7 mm to (209.1, 67.6), turned to 270 degrees
- moved C25 246.6 mm to (203.3, 60.2), turned to 270 degrees
- moved R2 246.3 mm to (211.0, 67.6), turned to 270 degrees
- moved U6 237.5 mm to (212.9, 57.3), turned to 270 degrees
- moved C26 233.1 mm to (210.0, 47.6), turned to 180 degrees
- moved BT1 226.9 mm to (212.4, 39.7), turned to 0 degrees
- moved AE1 164.2 mm to (202.0, 123.4), turned to 90 degrees
- moved C14 158.0 mm to (207.1, 127.8), turned to 90 degrees
- moved J14 155.9 mm to (206.2, 122.9), turned to 180 degrees
- moved U3 141.3 mm to (217.6, 130.4), turned to 180 degrees
- moved R29 76.9 mm to (82.6, 118.0), turned to 270 degrees
- moved R30 76.4 mm to (84.5, 118.0), turned to 90 degrees
- moved U1 7.50 mm to (132.2, 97.1)
Routing:
- net Net-(J16-Pad2): track 0.00 -> 9.24 mm
- net /VBAT2: track 0.00 -> 1.88 mm
- net GND: track 216.6 -> 218.3 mm
