File: Draco.kicad_pcb (KiCad board)
At the start: 2 copper layers, 95.2 x 44.5 mm, 117 parts, among them J1 Conn_01x03, J10 Conn_01x03, J11 Conn_01x06, J12 Conn_02x05_Odd_Even, J13 Conn_01x04, J14 Conn_01x01, J15 Micro_SD_Card, J16 Conn_01x03, J17 CHARGE_A, J18 CHARGE_C, J19 CHARGE_B, J2 Conn_01x03, J20 Conn_01x04, J3 Conn_01x03, J4 Conn_01x03, J5 Conn_01x03, J6 Conn_01x03, J7 Conn_01x03, J8 Conn_01x03, J9 Conn_01x03, Q1 BC817, Q2 Q_NMOS_DGS, Q3 BC817, Q4 Q_NMOS_DGS, Q5 BC817, Q6 Q_NMOS_DGS, U1 ATMEGA2560-16AU, U2 LOGIC-TXS0108EPWR(TSSOP20), U3 RFM95HW, U4 TPS54332, U5 TLV62568, U6 SAM-M8Q, U7 BMX055, U8 MS5607, Y1 16MHz

Commit message: Routed 50%
Parts:
- AE1, C14, J14, U2, U3: moved to B.Cu
- J11: footprint Connectors_JST:JST_PH_B6B-PH-K_06x2.00mm_Straight -> Socket_Strips:Socket_Strip_Straight_1x06_Pitch2.54mm
- J13: footprint Connectors_JST:JST_PH_B4B-PH-K_04x2.00mm_Straight -> Connectors_JST:JST_XH_B04B-XH-A_04x2.50mm_Straight
- J20: footprint Pin_Headers:Pin_Header_Angled_1x04_Pitch2.54mm -> Connectors_JST:JST_XH_B04B-XH-A_04x2.50mm_Straight
- moved J15 414.3 mm to (158.1, 113.2), turned to 180 degrees
- moved C13 411.0 mm to (156.8, 104.8), turned to 180 degrees
- moved J12 329.4 mm to (119.6, 89.5), turned to 180 degrees
- moved C7 326.2 mm to (129.9, 81.9), turned to 90 degrees
- moved J11 321.0 mm to (130.8, 78.3), turned to 90 degrees
- moved R8 276.2 mm to (124.2, 83.3), turned to 270 degrees
- moved R7 273.9 mm to (126.0, 83.3), turned to 270 degrees
- moved D3 271.9 mm to (124.2, 79.7), turned to 270 degrees
- moved R4 271.6 mm to (127.9, 83.3), turned to 270 degrees
- moved D2 269.6 mm to (126.0, 79.7), turned to 270 degrees
- moved D1 267.3 mm to (127.9, 79.7), turned to 270 degrees
- moved C12 219.6 mm to (241.0, 23.4)
- moved R11 198.7 mm to (165.3, 84.1), turned to 270 degrees
- moved R10 194.9 mm to (167.3, 84.1), turned to 270 degrees
- moved R9 191.1 mm to (169.4, 84.1), turned to 270 degrees
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Connections:
- R10 pad 2: /CAM_PWR -> /CAM_PHOTO
- R11 pad 2: /CAM_PHOTO -> /CAM_PWR
- U2 pad 12: /5V_LORA_RST -> /5V_MISO
- U2 pad 13: /5V_SD_NSS -> /5V_MOSI
- U2 pad 14: /5V_LORA_NSS -> /5V_SCK
- U2 pad 15: /5V_SCK -> /5V_LORA_NSS
- U2 pad 16: /5V_MISO -> /5V_LORA_RST
- U2 pad 17: /5V_MOSI -> /5V_SD_NSS
- U2 pad 4: /3V_MOSI -> /3V_SD_NSS
- U2 pad 5: /3V_MISO -> /3V_LORA_RST
- U2 pad 6: /3V_SCK -> /3V_LORA_NSS
- U2 pad 7: /3V_LORA_NSS -> /3V_SCK
- U2 pad 8: /3V_SD_NSS -> /3V_MOSI
- U2 pad 9: /3V_LORA_RST -> /3V_MISO
Routing:
- net GND: track 218.3 -> 333.4 mm, vias 0 -> 7
- net /RESET: track 0.00 -> 45.8 mm, vias 0 -> 3
- net /5V_MISO: track 0.00 -> 30.8 mm, vias 0 -> 2
- net /SERVO1: track 0.91 -> 30.1 mm, vias 0 -> 1
- net /5V_SCK: track 0.00 -> 27.4 mm
- net /SERVO2: track 0.03 -> 26.5 mm
- net Net-(C5-Pad1): track 0.00 -> 26.2 mm
- net /SERVO3: track 0.13 -> 23.8 mm
- net /PROG_RX: track 0.00 -> 23.0 mm
- net /PROG_TX: track 0.00 -> 22.8 mm
- net Net-(J1-Pad2): track 52.9 -> 30.8 mm
- net /5V_MOSI: track 0.00 -> 21.6 mm
- net /LED_GREEN: track 0.00 -> 20.8 mm
- net /LED_YELLOW: track 0.00 -> 20.6 mm
- net /SERVO4: track 0.13 -> 20.6 mm
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Other:
- board size 95.2 x 44.5 mm -> 114.3 x 44.5 mm
