File: Draco.kicad_pcb (KiCad board)
At the start: 2 copper layers, 114.3 x 44.5 mm, 122 parts, among them J1 Conn_01x03, J10 Conn_01x03, J11 Conn_01x06, J12 Conn_02x05_Odd_Even, J13 Conn_01x04, J14 Conn_01x01, J15 Micro_SD_Card, J16 Conn_01x03, J17 CHARGE_A, J18 CHARGE_C, J19 CHARGE_B, J2 Conn_01x03, J20 Conn_01x04, J3 Conn_01x03, J4 Conn_01x03, J5 Conn_01x03, J6 Conn_01x03, J7 Conn_01x03, J8 Conn_01x03, J9 Conn_01x03, Q1 BC817, Q2 Q_NMOS_DGS, Q3 BC817, Q4 Q_NMOS_DGS, Q5 BC817, Q6 Q_NMOS_DGS, U1 ATMEGA2560-16AU, U2 LOGIC-TXS0108EPWR(TSSOP20), U3 RFM95HW, U4 TPS54332, U5 TLV62568, U6 SAM-M8Q, U7 LSM9DS1TR‎, U8 MS5607, Y1 16MHz

Commit message: Finished preliminary layout
Parts:
- C1, C2, C25, C26, C27, C3, C6: moved to B.Cu
- moved C28 131.6 mm to (180.6, 78.7)
- moved C26 118.6 mm to (176.7, 91.5)
- moved C25 109.6 mm to (164.2, 108.0), turned to 270 degrees
- moved C27 90.9 mm to (150.9, 113.9), turned to 270 degrees
- moved C3 81.6 mm to (135.8, 89.2), turned to 90 degrees
- moved C2 44.9 mm to (106.7, 118.5), turned to 270 degrees
- moved C1 44.1 mm to (108.5, 118.5), turned to 270 degrees
- moved C6 39.6 mm to (103.2, 113.1), turned to 90 degrees
Connections:
- J11 pad 5: Net-(J11-Pad5) -> (no net)
- J12 pad 3: Net-(J12-Pad3) -> (no net)
- J15 pad 1: Net-(J15-Pad1) -> (no net)
- J15 pad 8: Net-(J15-Pad8) -> (no net)
- U1 pad 1: Net-(U1-Pad1) -> (no net)
- U1 pad 12: Net-(U1-Pad12) -> (no net)
- U1 pad 13: Net-(U1-Pad13) -> (no net)
- U1 pad 14: Net-(U1-Pad14) -> (no net)
- U1 pad 18: Net-(U1-Pad18) -> (no net)
- U1 pad 19: Net-(U1-Pad19) -> (no net)
- U1 pad 23: Net-(U1-Pad23) -> (no net)
- U1 pad 24: Net-(U1-Pad24) -> (no net)
- U1 pad 25: Net-(U1-Pad25) -> (no net)
- U1 pad 26: Net-(U1-Pad26) -> (no net)
- U1 pad 27: Net-(U1-Pad27) -> (no net)
- U1 pad 28: Net-(U1-Pad28) -> (no net)
- U1 pad 29: Net-(U1-Pad29) -> (no net)
- U1 pad 4: Net-(U1-Pad4) -> (no net)
- U1 pad 47: Net-(U1-Pad47) -> (no net)
- U1 pad 48: Net-(U1-Pad48) -> (no net)
- U1 pad 49: Net-(U1-Pad49) -> (no net)
- U1 pad 5: Net-(U1-Pad5) -> (no net)
- U1 pad 50: Net-(U1-Pad50) -> (no net)
- U1 pad 51: Net-(U1-Pad51) -> (no net)
- U1 pad 52: Net-(U1-Pad52) -> (no net)
- U1 pad 53: Net-(U1-Pad53) -> (no net)
- U1 pad 54: Net-(U1-Pad54) -> (no net)
- U1 pad 55: Net-(U1-Pad55) -> (no net)
- U1 pad 56: Net-(U1-Pad56) -> (no net)
- U1 pad 57: Net-(U1-Pad57) -> (no net)
- U1 pad 58: Net-(U1-Pad58) -> (no net)
- U1 pad 59: Net-(U1-Pad59) -> (no net)
- U1 pad 60: Net-(U1-Pad60) -> (no net)
- U1 pad 63: Net-(U1-Pad63) -> (no net)
- U1 pad 64: Net-(U1-Pad64) -> (no net)
- U1 pad 65: Net-(U1-Pad65) -> (no net)
- U1 pad 69: Net-(U1-Pad69) -> (no net)
- U1 pad 70: Net-(U1-Pad70) -> (no net)
- U1 pad 79: Net-(U1-Pad79) -> (no net)
- U1 pad 84: Net-(U1-Pad84) -> (no net)
- U1 pad 85: Net-(U1-Pad85) -> (no net)
- U1 pad 86: Net-(U1-Pad86) -> (no net)
- U1 pad 90: Net-(U1-Pad90) -> (no net)
- U1 pad 91: Net-(U1-Pad91) -> (no net)
- U3 pad 11: Net-(U3-Pad11) -> (no net)
- U3 pad 12: Net-(U3-Pad12) -> (no net)
- U3 pad 15: Net-(U3-Pad15) -> (no net)
- U3 pad 16: Net-(U3-Pad16) -> (no net)
- U3 pad 7: Net-(U3-Pad7) -> (no net)
- U4 pad 3: Net-(U4-Pad3) -> (no net)
- U6 pad 18: Net-(U6-Pad18) -> (no net)
- U6 pad 7: Net-(U6-Pad7) -> (no net)
- U6 pad 8: Net-(U6-Pad8) -> (no net)
- U7 pad 10: Net-(U7-Pad10) -> (no net)
- U7 pad 13: Net-(U7-Pad13) -> (no net)
- U7 pad 5: Net-(U7-Pad5) -> (no net)
- U7 pad 6: Net-(U7-Pad6) -> (no net)
Routing:
- net GND: track 541.2 -> 570.1 mm, vias 21 -> 22
- net +5V: track 198.9 -> 215.6 mm, vias 5 -> 8
- net +3V3: track 210.5 -> 215.9 mm, vias 10 -> 11
Other:
- board text added: "Draco_Rev1 Rocket Control Board By Vlad Pomogaev"
