File: power.sch (KiCad schematic (older format))
At the start: 18 parts, among them J14 Conn_01x02, U3 LM2574-5.0V, U4 LM2574-3.3V

Commit message: Did design review. Changed/confirmed voltage levels
Parts:
- removed D1: D, symbol D
- added D4: B0520LW-7-F, symbol D_Schottky
- added JP2: Jumper_NO_Small, symbol Jumper_NO_Small
- C15: renamed from C13; footprint (none) -> Capacitors_SMD:C_0805
- C16: renamed from C14; footprint (none) -> Capacitors_SMD:C_0805
- C18: renamed from C16; footprint (none) -> Capacitors_SMD:C_0805
- C20: renamed from C18; footprint (none) -> Capacitors_SMD:C_0805
- C23: renamed from C21; footprint (none) -> Capacitors_SMD:C_0805
- C24: renamed from C22; footprint (none) -> Capacitors_SMD:C_0805
- renumbered C15 to C17, C17 to C19, C19 to C21, C20 to C22, D2 to D5, D3 to D6, J14 to J16, U3 to U4, U4 to U5
Connections:
- net +BATT: now also D4.2 (A), JP2.2; no longer J16.1 (Pin_1)
- net at U4.10 (VIN): now also D4.1 (K)
- new net VCC: J16.1 (Pin_1), JP2.1
Other:
- moved on the sheet: J16
Changed lines of the file:
@@
 $EndDescr
 $Comp
-L Conn_01x02 J14
+L Conn_01x02 J16
 U 1 1 5A59B267
-P 2900 2400
-F 0 "J14" H 2900 2500 50  0000 C CNN
-F 1 "Conn_01x02" H 2900 2200 50  0000 C CNN
-F 2 "" H 2900 2400 50  0001 C CNN
-F 3 "" H 2900 2400 50  0001 C CNN
-	1    2900 2400
-	-1   0    0    -1
-$EndComp
-$Comp
-L GND #PWR024
+P 2500 2400
+F 0 "J16" H 2500 2500 50  0000 C CNN
+F 1 "Conn_01x02" H 2500 2200 50  0000 C CNN
+F 2 "" H 2500 2400 50  0001 C CNN
+F 3 "" H 2500 2400 50  0001 C CNN
+	1    2500 2400
+	-1   0    0    -1
+$EndComp
+$Comp
+L GND #PWR034
 U 1 1 5A59B2D2
-P 3250 2650
-F 0 "#PWR024" H 3250 2400 50  0001 C CNN
-F 1 "GND" H 3250 2500 50  0000 C CNN
-F 2 "" H 3250 2650 50  0001 C CNN
-F 3 "" H 3250 2650 50  0001 C CNN
-	1    3250 2650
-	1    0    0    -1
-$EndComp
-$Comp
-L C C13
+P 2850 2650
+F 0 "#PWR034" H 2850 2400 50  0001 C CNN
+F 1 "GND" H 2850 2500 50  0000 C CNN
+F 2 "" H 2850 2650 50  0001 C CNN
+F 3 "" H 2850 2650 50  0001 C CNN
+	1    2850 2650
+	1    0    0    -1
+$EndComp
+$Comp
+L C C15
 U 1 1 5A59B2FE
 P 3500 2650
-F 0 "C13" H 3525 2750 50  0000 L CNN
+F 0 "C15" H 3525 2750 50  0000 L CNN
 F 1 "100nF" H 3525 2550 50  0000 L CNN
-F 2 "" H 3538 2500 50  0001 C CNN
+F 2 "Capacitors_SMD:C_0805" H 3538 2500 50  0001 C CNN
 F 3 "" H 3500 2650 50  0001 C CNN
 	1    3500 2650
@@
 $EndComp
 $Comp
-L GND #PWR025
+L GND #PWR035
 U 1 1 5A59B35D
 P 3500 3000
-F 0 "#PWR025" H 3500 2750 50  0001 C CNN
+F 0 "#PWR035" H 3500 2750 50  0001 C CNN
 F 1 "GND" H 3500 2850 50  0000 C CNN
 F 2 "" H 3500 3000 50  0001 C CNN
@@
 $EndComp
 $Comp
-L +BATT #PWR026
+L +BATT #PWR036
 U 1 1 5A5B961D
 P 3250 2250
-F 0 "#PWR026" H 3250 2100 50  0001 C CNN
+F 0 "#PWR036" H 3250 2100 50  0001 C CNN
 F 1 "+BATT" H 3250 2390 50  0000 C CNN
 F 2 "" H 3250 2250 50  0001 C CNN
@@
 $EndComp
 $Comp
-L C C14
+L C C16
 U 1 1 5A5BA8AA
 P 3850 2650
-F 0 "C14" H 3875 2750 50  0000 L CNN
+F 0 "C16" H 3875 2750 50  0000 L CNN
 F 1 "100nF" H 3875 2550 50  0000 L CNN
-F 2 "" H 3888 2500 50  0001 C CNN
+F 2 "Capacitors_SMD:C_0805" H 3888 2500 50  0001 C CNN
 F 3 "" H 3850 2650 50  0001 C CNN
 	1    3850 2650
@@
 $EndComp
 $Comp
-L CP C15
+L CP C17
 U 1 1 5A5BA8CA
 P 4200 2650
-F 0 "C15" H 4225 2750 50  0000 L CNN
+F 0 "C17" H 4225 2750 50  0000 L CNN
 F 1 "22uF" H 4225 2550 50  0000 L CNN
 F 2 "" H 4238 2500 50  0001 C CNN
@@
 $EndComp
 $Comp
-L LM2574 U3
+L LM2574 U4
 U 1 1 5A5BB86F
 P 5700 2700
-F 0 "U3" H 5250 3250 60  0000 L CNN
+F 0 "U4" H 5250 3250 60  0000 L CNN
 F 1 "LM2574-5.0V" H 5250 3150 60  0000 L CNN
 F 2 "" H 5700 2700 60  0001 C CNN
@@
 $EndComp
 Wire Wire Line
-	3100 2500 3250 2500
-Wire Wire Line
-	3250 2500 3250 2650
-Wire Wire Line
-	3100 2400 4750 2400
+	2700 2500 2850 2500
+Wire Wire Line
+	2850 2500 2850 2650
+Wire Wire Line
+	3000 2400 4750 2400
 Wire Wire Line
 	3500 2400 3500 2500
@@
 Connection ~ 5700 3250
 $Comp
-L GND #PWR027
+L GND #PWR037
 U 1 1 5A5BC20B
 P 5700 3350
-F 0 "#PWR027" H 5700 3100 50  0001 C CNN
+F 0 "#PWR037" H 5700 3100 50  0001 C CNN
 F 1 "GND" H 5700 3200 50  0000 C CNN
 F 2 "" H 5700 3350 50  0001 C CNN
@@
 $EndComp
 $Comp
-L CP C20
+L CP C22
 U 1 1 5A5BC236
 P 7500 2800
-F 0 "C20" H 7525 2900 50  0000 L CNN
+F 0 "C22" H 7525 2900 50  0000 L CNN
 F 1 "200uF" H 7525 2700 50  0000 L CNN
 F 2 "" H 7538 2650 50  0001 C CNN
@@
 $EndComp
 $Comp
-L D_Schottky D3
+L D_Schottky D6
 U 1 1 5A5BC3C5
 P 6600 2800
-F 0 "D3" H 6600 2900 50  0000 C CNN
+F 0 "D6" H 6600 2900 50  0000 C CNN
 F 1 "11DQ06" H 6600 2700 50  0000 C CNN
 F 2 "" H 6600 2800 50  0001 C CNN
@@
 	7500 2950 7500 3050
 $Comp
-L GND #PWR028
+L GND #PWR038
 U 1 1 5A5BC575
 P 6600 3050
-F 0 "#PWR028" H 6600 2800 50  0001 C CNN
+F 0 "#PWR038" H 6600 2800 50  0001 C CNN
 F 1 "GND" H 6600 2900 50  0000 C CNN
 F 2 "" H 6600 3050 50  0001 C CNN
@@
 $EndComp
 $Comp
-L GND #PWR029
+L GND #PWR039
 U 1 1 5A5BC598
 P 7500 3050
-F 0 "#PWR029" H 7500 2800 50  0001 C CNN
+F 0 "#PWR039" H 7500 2800 50  0001 C CNN
 F 1 "GND" H 7500 2900 50  0000 C CNN
 F 2 "" H 7500 3050 50  0001 C CNN
@@
 	8400 2400 8400 3900
 $Comp
-L +5V #PWR030
+L +5V #PWR040
 U 1 1 5A5BC607
 P 8400 2400
-F 0 "#PWR030" H 8400 2250 50  0001 C CNN
+F 0 "#PWR040" H 8400 2250 50  0001 C CNN
 F 1 "+5V" H 8400 2540 50  0000 C CNN
 F 2 "" H 8400 2400 50  0001 C CNN
@@
 $EndComp
 $Comp
-L LM2574 U4
+L LM2574 U5
 U 1 1 5A5BCA9B
 P 6650 4200
-F 0 "U4" H 6200 4750 60  0000 L CNN
+F 0 "U5" H 6200 4750 60  0000 L CNN
 F 1 "LM2574-3.3V" H 6200 4650 60  0000 L CNN
 F 2 "" H 6650 4200 60  0001 C CNN
@@
 Connection ~ 6650 4750
 $Comp
-L GND #PWR031
+L GND #PWR041
 U 1 1 5A5BCAA7
 P 6650 4850
-F 0 "#PWR031" H 6650 4600 50  0001 C CNN
+F 0 "#PWR041" H 6650 4600 50  0001 C CNN
 F 1 "GND" H 6650 4700 50  0000 C CNN
 F 2 "" H 6650 4850 50  0001 C CNN
@@
 $EndComp
 $Comp
-L CP C19
+L CP C21
 U 1 1 5A5BCAAD
 P 4850 4300
-F 0 "C19" H 4875 4400 50  0000 L CNN
+F 0 "C21" H 4875 4400 50  0000 L CNN
 F 1 "200uF" H 4875 4200 50  0000 L CNN
 F 2 "" H 4888 4150 50  0001 C CNN
@@
 $EndComp
 $Comp
-L D_Schottky D2
+L D_Schottky D5
 U 1 1 5A5BCAB9
 P 5750 4300
-F 0 "D2" H 5750 4400 50  0000 C CNN
+F 0 "D5" H 5750 4400 50  0000 C CNN
 F 1 "11DQ06" H 5750 4200 50  0000 C CNN
 F 2 "" H 5750 4300 50  0001 C CNN
@@
 	4850 4450 4850 4550
 $Comp
-L GND #PWR032
+L GND #PWR042
 U 1 1 5A5BCAC6
 P 5750 4550
-F 0 "#PWR032" H 5750 4300 50  0001 C CNN
+F 0 "#PWR042" H 5750 4300 50  0001 C CNN
 F 1 "GND" H 5750 4400 50  0000 C CNN
 F 2 "" H 5750 4550 50  0001 C CNN
@@
 $EndComp
 $Comp
-L GND #PWR033
+L GND #PWR043
 U 1 1 5A5BCACC
 P 4850 4550
-F 0 "#PWR033" H 4850 4300 50  0001 C CNN
+F 0 "#PWR043" H 4850 4300 50  0001 C CNN
 F 1 "GND" H 4850 4400 50  0000 C CNN
 F 2 "" H 4850 4550 50  0001 C CNN
@@
 	8400 3900 7300 3900
 $Comp
-L +3.3V #PWR034
+L +3.3V #PWR044
 U 1 1 5A5BCDF5
 P 3950 3900
-F 0 "#PWR034" H 3950 3750 50  0001 C CNN
+F 0 "#PWR044" H 3950 3750 50  0001 C CNN
 F 1 "+3.3V" H 3950 4040 50  0000 C CNN
 F 2 "" H 3950 3900 50  0001 C CNN
@@
 $EndComp
 $Comp
-L CP C17
+L CP C19
 U 1 1 5A5BD7F7
 P 4500 2650
-F 0 "C17" H 4525 2750 50  0000 L CNN
+F 0 "C19" H 4525 2750 50  0000 L CNN
 F 1 "22uF" H 4525 2550 50  0000 L CNN
 F 2 "" H 4538 2500 50  0001 C CNN
@@
 Connection ~ 4200 2900
 $Comp
-L C C18
+L C C20
 U 1 1 5A5D30DE
 P 4500 4300
-F 0 "C18" H 4525 4400 50  0000 L CNN
+F 0 "C20" H 4525 4400 50  0000 L CNN
 F 1 "100nF" H 4525 4200 50  0000 L CNN
-F 2 "" H 4538 4150 50  0001 C CNN
+F 2 "Capacitors_SMD:C_0805" H 4538 4150 50  0001 C CNN
 F 3 "" H 4500 4300 50  0001 C CNN
 	1    4500 4300
@@
 $EndComp
 $Comp
-L C C16
+L C C18
 U 1 1 5A5D316B
 P 4200 4300
-F 0 "C16" H 4225 4400 50  0000 L CNN
+F 0 "C18" H 4225 4400 50  0000 L CNN
 F 1 "100nF" H 4225 4200 50  0000 L CNN
-F 2 "" H 4238 4150 50  0001 C CNN
+F 2 "Capacitors_SMD:C_0805" H 4238 4150 50  0001 C CNN
 F 3 "" H 4200 4300 50  0001 C CNN
 	1    4200 4300
@@
 $EndComp
 $Comp
-L C C21
+L C C23
 U 1 1 5A5D31B4
 P 7850 2800
-F 0 "C21" H 7875 2900 50  0000 L CNN
+F 0 "C23" H 7875 2900 50  0000 L CNN
 F 1 "100nF" H 7875 2700 50  0000 L CNN
-F 2 "" H 7888 2650 50  0001 C CNN
+F 2 "Capacitors_SMD:C_0805" H 7888 2650 50  0001 C CNN
 F 3 "" H 7850 2800 50  0001 C CNN
 	1    7850 2800
@@
 $EndComp
 $Comp
-L C C22
+L C C24
 U 1 1 5A5D3210
 P 8150 2800
-F 0 "C22" H 8175 2900 50  0000 L CNN
+F 0 "C24" H 8175 2900 50  0000 L CNN
 F 1 "100nF" H 8175 2700 50  0000 L CNN
-F 2 "" H 8188 2650 50  0001 C CNN
+F 2 "Capacitors_SMD:C_0805" H 8188 2650 50  0001 C CNN
 F 3 "" H 8150 2800 50  0001 C CNN
 	1    8150 2800
@@
 	8150 2650 8150 2550
 Connection ~ 8150 2550
-$Comp
-L D D1
-U 1 1 5A5DA963
+Connection ~ 8400 2550
+$Comp
+L D_Schottky D4
+U 1 1 5A660E68
 P 4900 2400
-F 0 "D1" H 4900 2500 50  0000 C CNN
-F 1 "D" H 4900 2300 50  0000 C CNN
+F 0 "D4" H 4900 2500 50  0000 C CNN
+F 1 "B0520LW-7-F" H 4900 2300 50  0000 C CNN
 F 2 "" H 4900 2400 50  0001 C CNN
 F 3 "" H 4900 2400 50  0001 C CNN
@@
 	-1   0    0    1
 $EndComp
-Connection ~ 8400 2550
+$Comp
+L Jumper_NO_Small JP2
+U 1 1 5A68672B
+P 2900 2400
+F 0 "JP2" H 2900 2480 50  0000 C CNN
+F 1 "Jumper_NO_Small" H 2910 2340 50  0000 C CNN
+F 2 "" H 2900 2400 50  0001 C CNN
+F 3 "" H 2900 2400 50  0001 C CNN
+	1    2900 2400
+	1    0    0    -1
+$EndComp
+Wire Wire Line
+	2800 2400 2700 2400
+$Comp
+L VCC #PWR045
+U 1 1 5A686A35
+P 2750 2250
+F 0 "#PWR045" H 2750 2100 50  0001 C CNN
+F 1 "VCC" H 2750 2400 50  0000 C CNN
+F 2 "" H 2750 2250 50  0001 C CNN
+F 3 "" H 2750 2250 50  0001 C CNN
+	1    2750 2250
+	1    0    0    -1
+$EndComp
+Wire Wire Line
+	2750 2400 2750 2250
+Connection ~ 2750 2400
 $EndSCHEMATC

Commit message: Started Board layout
Parts:
- removed J16: Conn_01x02, symbol Conn_01x02
- added J16: Conn_01x03, Connectors_JST:JST_XH_S03B-XH-A_03x2.50mm_Angled, symbol Conn_01x03
- added R29, R30: 10K, Resistors_SMD:R_0805, symbol R
- C17, C19, C21, C22: footprint (none) -> Capacitors_THT:CP_Radial_D5.0mm_P2.00mm
- D4: footprint (none) -> Diodes_SMD:D_SOD-123
- D5, D6: footprint (none) -> Diodes_THT:D_DO-41_SOD81_P2.54mm_Vertical_AnodeUp
- JP2: footprint (none) -> Pin_Headers:Pin_Header_Straight_1x02_Pitch2.54mm
- L2: value 330uF 1A -> 100uH 0.5A; footprint (none) -> Inductors_THT:L_Radial_D8.7mm_P5.00mm_Fastron_07HCP
- L3: footprint (none) -> Inductors_THT:L_Radial_D8.7mm_P5.00mm_Fastron_07HCP
- U4, U5: footprint (none) -> Housings_SOIC:SOIC-14W_7.5x9.0mm_Pitch1.27mm
Connections:
- net GND: now also J16.3 (Pin_3), R30.2
- net VCC: now also J16.1 (Pin_1)
- new net: J16.2 (Pin_2), R29.1
- new net VBAT2: R29.2, R30.1
Changed lines of the file:
@@
 LIBS:TXB0104DR
 LIBS:LOGIC-TXS0108EPWR_TSSOP20_
+LIBS:CurrentControlSystems
 LIBS:Draco-cache
 EELAYER 25 0
@@
 $EndDescr
 $Comp
-L Conn_01x02 J16
-U 1 1 5A59B267
-P 2500 2400
-F 0 "J16" H 2500 2500 50  0000 C CNN
-F 1 "Conn_01x02" H 2500 2200 50  0000 C CNN
-F 2 "" H 2500 2400 50  0001 C CNN
-F 3 "" H 2500 2400 50  0001 C CNN
-	1    2500 2400
-	-1   0    0    -1
-$EndComp
-$Comp
 L GND #PWR034
 U 1 1 5A59B2D2
-P 2850 2650
-F 0 "#PWR034" H 2850 2400 50  0001 C CNN
-F 1 "GND" H 2850 2500 50  0000 C CNN
-F 2 "" H 2850 2650 50  0001 C CNN
-F 3 "" H 2850 2650 50  0001 C CNN
-	1    2850 2650
+P 2800 2750
+F 0 "#PWR034" H 2800 2500 50  0001 C CNN
+F 1 "GND" H 2800 2600 50  0000 C CNN
+F 2 "" H 2800 2750 50  0001 C CNN
+F 3 "" H 2800 2750 50  0001 C CNN
+	1    2800 2750
 	1    0    0    -1
 $EndComp
@@
 F 0 "C17" H 4225 2750 50  0000 L CNN
 F 1 "22uF" H 4225 2550 50  0000 L CNN
-F 2 "" H 4238 2500 50  0001 C CNN
+F 2 "Capacitors_THT:CP_Radial_D5.0mm_P2.00mm" H 4238 2500 50  0001 C CNN
 F 3 "" H 4200 2650 50  0001 C CNN
 	1    4200 2650
 	1    0    0    -1
 $EndComp
-$Comp
-L LM2574 U4
-U 1 1 5A5BB86F
-P 5700 2700
-F 0 "U4" H 5250 3250 60  0000 L CNN
-F 1 "LM2574-5.0V" H 5250 3150 60  0000 L CNN
-F 2 "" H 5700 2700 60  0001 C CNN
-F 3 "" H 5700 2700 60  0001 C CNN
-	1    5700 2700
-	1    0    0    -1
-$EndComp
-Wire Wire Line
-	2700 2500 2850 2500
-Wire Wire Line
-	2850 2500 2850 2650
+Wire Wire Line
+	2500 2600 2800 2600
+Wire Wire Line
+	2800 2600 2800 2750
 Wire Wire Line
 	3000 2400 4750 2400
@@
 F 0 "C22" H 7525 2900 50  0000 L CNN
 F 1 "200uF" H 7525 2700 50  0000 L CNN
-F 2 "" H 7538 2650 50  0001 C CNN
+F 2 "Capacitors_THT:CP_Radial_D5.0mm_P2.00mm" H 7538 2650 50  0001 C CNN
 F 3 "" H 7500 2800 50  0001 C CNN
 	1    7500 2800
@@
 F 0 "L3" V 6950 2550 50  0000 C CNN
 F 1 "330uF 1A" V 7075 2550 50  0000 C CNN
-F 2 "" H 7000 2550 50  0001 C CNN
+F 2 "Inductors_THT:L_Radial_D8.7mm_P5.00mm_Fastron_07HCP" H 7000 2550 50  0001 C CNN
 F 3 "" H 7000 2550 50  0001 C CNN
 	1    7000 2550
@@
 F 0 "D6" H 6600 2900 50  0000 C CNN
 F 1 "11DQ06" H 6600 2700 50  0000 C CNN
-F 2 "" H 6600 2800 50  0001 C CNN
+F 2 "Diodes_THT:D_DO-41_SOD81_P2.54mm_Vertical_AnodeUp" H 6600 2800 50  0001 C CNN
 F 3 "" H 6600 2800 50  0001 C CNN
 	1    6600 2800
@@
 	1    0    0    -1
 $EndComp
-$Comp
-L LM2574 U5
-U 1 1 5A5BCA9B
-P 6650 4200
-F 0 "U5" H 6200 4750 60  0000 L CNN
-F 1 "LM2574-3.3V" H 6200 4650 60  0000 L CNN
-F 2 "" H 6650 4200 60  0001 C CNN
-F 3 "" H 6650 4200 60  0001 C CNN
-	1    6650 4200
-	-1   0    0    -1
-$EndComp
 Wire Wire Line
 	6800 4750 6800 4700
@@
 F 0 "C21" H 4875 4400 50  0000 L CNN
 F 1 "200uF" H 4875 4200 50  0000 L CNN
-F 2 "" H 4888 4150 50  0001 C CNN
+F 2 "Capacitors_THT:CP_Radial_D5.0mm_P2.00mm" H 4888 4150 50  0001 C CNN
 F 3 "" H 4850 4300 50  0001 C CNN
 	1    4850 4300
@@
 P 5350 4050
 F 0 "L2" V 5300 4050 50  0000 C CNN
-F 1 "330uF 1A" V 5425 4050 50  0000 C CNN
-F 2 "" H 5350 4050 50  0001 C CNN
+F 1 "100uH 0.5A" V 5425 4050 50  0000 C CNN
+F 2 "Inductors_THT:L_Radial_D8.7mm_P5.00mm_Fastron_07HCP" H 5350 4050 50  0001 C CNN
 F 3 "" H 5350 4050 50  0001 C CNN
 	1    5350 4050
@@
 F 0 "D5" H 5750 4400 50  0000 C CNN
 F 1 "11DQ06" H 5750 4200 50  0000 C CNN
-F 2 "" H 5750 4300 50  0001 C CNN
+F 2 "Diodes_THT:D_DO-41_SOD81_P2.54mm_Vertical_AnodeUp" H 5750 4300 50  0001 C CNN
 F 3 "" H 5750 4300 50  0001 C CNN
 	1    5750 4300
@@
 F 0 "C19" H 4525 2750 50  0000 L CNN
 F 1 "22uF" H 4525 2550 50  0000 L CNN
-F 2 "" H 4538 2500 50  0001 C CNN
+F 2 "Capacitors_THT:CP_Radial_D5.0mm_P2.00mm" H 4538 2500 50  0001 C CNN
 F 3 "" H 4500 2650 50  0001 C CNN
 	1    4500 2650
@@
 F 0 "D4" H 4900 2500 50  0000 C CNN
 F 1 "B0520LW-7-F" H 4900 2300 50  0000 C CNN
-F 2 "" H 4900 2400 50  0001 C CNN
+F 2 "Diodes_SMD:D_SOD-123" H 4900 2400 50  0001 C CNN
 F 3 "" H 4900 2400 50  0001 C CNN
 	1    4900 2400
@@
 F 0 "JP2" H 2900 2480 50  0000 C CNN
 F 1 "Jumper_NO_Small" H 2910 2340 50  0000 C CNN
-F 2 "" H 2900 2400 50  0001 C CNN
+F 2 "Pin_Headers:Pin_Header_Straight_1x02_Pitch2.54mm" H 2900 2400 50  0001 C CNN
 F 3 "" H 2900 2400 50  0001 C CNN
 	1    2900 2400
@@
 $EndComp
 Wire Wire Line
-	2800 2400 2700 2400
+	2500 2400 2800 2400
 $Comp
 L VCC #PWR045
@@
 	2750 2400 2750 2250
 Connection ~ 2750 2400
+$Comp
+L LM2574 U5
+U 1 1 5A5BCA9B
+P 6650 4200
+F 0 "U5" H 6200 4750 60  0000 L CNN
+F 1 "LM2574-3.3V" H 6200 4650 60  0000 L CNN
+F 2 "Housings_SOIC:SOIC-14W_7.5x9.0mm_Pitch1.27mm" H 6650 4200 60  0001 C CNN
+F 3 "" H 6650 4200 60  0001 C CNN
+	1    6650 4200
+	-1   0    0    -1
+$EndComp
+$Comp
+L LM2574 U4
+U 1 1 5A5BB86F
+P 5700 2700
+F 0 "U4" H 5250 3250 60  0000 L CNN
+F 1 "LM2574-5.0V" H 5250 3150 60  0000 L CNN
+F 2 "Housings_SOIC:SOIC-14W_7.5x9.0mm_Pitch1.27mm" H 5700 2700 60  0001 C CNN
+F 3 "" H 5700 2700 60  0001 C CNN
+	1    5700 2700
+	1    0    0    -1
+$EndComp
+$Comp
+L Conn_01x03 J16
+U 1 1 5A659ED4
+P 2300 2500
+F 0 "J16" H 2300 2700 50  0000 C CNN
+F 1 "Conn_01x03" H 2300 2300 50  0000 C CNN
+F 2 "Connectors_JST:JST_XH_S03B-XH-A_03x2.50mm_Angled" H 2300 2500 50  0001 C CNN
+F 3 "" H 2300 2500 50  0001 C CNN
+	1    2300 2500
+	-1   0    0    -1
+$EndComp
+Wire Wire Line
+	2500 2500 3150 2500
+Wire Wire Line
+	3150 2500 3150 3050
+$Comp
+L R R29
+U 1 1 5A65A109
+P 3150 3200
+F 0 "R29" V 3230 3200 50  0000 C CNN
+F 1 "10K" V 3150 3200 50  0000 C CNN
+F 2 "Resistors_SMD:R_0805" V 3080 3200 50  0001 C CNN
+F 3 "" H 3150 3200 50  0001 C CNN
+	1    3150 3200
+	1    0    0    -1
+$EndComp
+$Comp
+L R R30
+U 1 1 5A65A17C
+P 3150 3550
+F 0 "R30" V 3230 3550 50  0000 C CNN
+F 1 "10K" V 3150 3550 50  0000 C CNN
+F 2 "Resistors_SMD:R_0805" V 3080 3550 50  0001 C CNN
+F 3 "" H 3150 3550 50  0001 C CNN
+	1    3150 3550
+	1    0    0    -1
+$EndComp
+$Comp
+L GND #PWR046
+U 1 1 5A65A1D5
+P 3150 3750
+F 0 "#PWR046" H 3150 3500 50  0001 C CNN
+F 1 "GND" H 3150 3600 50  0000 C CNN
+F 2 "" H 3150 3750 50  0001 C CNN
+F 3 "" H 3150 3750 50  0001 C CNN
+	1    3150 3750
+	1    0    0    -1
+$EndComp
+Wire Wire Line
+	3150 3750 3150 3700
+Wire Wire Line
+	3150 3400 3150 3350
+Wire Wire Line
+	3150 3400 2950 3400
+Text HLabel 2950 3400 0    60   Output ~ 0
+VBAT2
 $EndSCHEMATC
