File: _saved_Draco.sch (KiCad schematic (older format))
At the start: 51 parts, among them J1 Conn_01x03, J10 Conn_01x03, J11 Conn_01x06, J12 Conn_02x05_Odd_Even, J13 Conn_01x04, J15 Micro_SD_Card, J2 Conn_01x03, J20 Conn_01x04, J3 Conn_01x03, J4 Conn_01x03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

Commit message: 80% done routing
Parts:
- J14: renamed from J?; footprint (none) -> Pin_Headers:Pin_Header_Straight_1x01_Pitch2.54mm
Other:
- moved on the sheet: AE1
Changed lines of the file:
@@
 L Antenna_Shield AE1
 U 1 1 5A5F375E
-P 14400 7150
-F 0 "AE1" H 14325 7325 50  0000 R CNN
-F 1 "Antenna_Shield" H 14325 7250 50  0000 R CNN
-F 2 "Current_Control_Systems:U.FL-R-SMT" H 14400 7250 50  0001 C CNN
-F 3 "" H 14400 7250 50  0001 C CNN
-	1    14400 7150
+P 14400 7100
+F 0 "AE1" H 14325 7275 50  0000 R CNN
+F 1 "Antenna_Shield" H 14325 7200 50  0000 R CNN
+F 2 "Current_Control_Systems:U.FL-R-SMT" H 14400 7200 50  0001 C CNN
+F 3 "" H 14400 7200 50  0001 C CNN
+	1    14400 7100
 	1    0    0    -1
 $EndComp
@@
 $EndComp
 Wire Wire Line
-	6350 7700 6350 7900
-Wire Wire Line
-	5950 7800 6350 7800
+	6350 7700 6350 7800
+Wire Wire Line
+	6350 7800 6350 7900
+Wire Wire Line
+	5950 7800 6050 7800
+Wire Wire Line
+	6050 7800 6150 7800
+Wire Wire Line
+	6150 7800 6250 7800
+Wire Wire Line
+	6250 7800 6350 7800
 Wire Wire Line
 	6250 7800 6250 7700
@@
 Connection ~ 6350 7800
 Wire Wire Line
-	5750 1700 5750 1900
-Wire Wire Line
-	5750 1800 6050 1800
+	5750 1700 5750 1800
+Wire Wire Line
+	5750 1800 5750 1900
+Wire Wire Line
+	5750 1800 5850 1800
+Wire Wire Line
+	5850 1800 5950 1800
+Wire Wire Line
+	5950 1800 6050 1800
 Wire Wire Line
 	6050 1800 6050 1900
@@
 Connection ~ 5750 1800
 Wire Wire Line
-	6250 1600 6250 1900
+	6250 1600 6250 1750
+Wire Wire Line
+	6250 1750 6250 1900
 Wire Wire Line
 	6250 1300 6250 1200
@@
 	6700 1750 6700 1850
 Wire Wire Line
-	4250 2500 4800 2500
-Wire Wire Line
-	4250 2800 4800 2800
+	4250 2500 4550 2500
+Wire Wire Line
+	4550 2500 4800 2500
+Wire Wire Line
+	4250 2800 4550 2800
+Wire Wire Line
+	4550 2800 4800 2800
 Connection ~ 4550 2500
 Connection ~ 4550 2800
@@
 	3950 2500 3800 2500
 Wire Wire Line
-	3800 2500 3800 2850
+	3800 2500 3800 2800
+Wire Wire Line
+	3800 2800 3800 2850
 Wire Wire Line
 	3800 2800 3950 2800
 Connection ~ 3800 2800
 Wire Wire Line
-	3800 2200 4800 2200
+	3800 2200 4350 2200
+Wire Wire Line
+	4350 2200 4650 2200
+Wire Wire Line
+	4650 2200 4800 2200
 Wire Wire Line
 	4650 2200 4650 2100
@@
 	10050 9150 10250 9150
 Wire Wire Line
-	10250 9150 10250 9650
+	10250 9150 10250 9250
+Wire Wire Line
+	10250 9250 10250 9350
+Wire Wire Line
+	10250 9350 10250 9450
+Wire Wire Line
+	10250 9450 10250 9650
 Wire Wire Line
 	10050 9450 10250 9450
@@
 	3150 9150 3150 9050
 Wire Wire Line
-	3150 9050 5250 9050
+	3150 9050 3500 9050
+Wire Wire Line
+	3500 9050 3850 9050
+Wire Wire Line
+	3850 9050 4050 9050
+Wire Wire Line
+	4050 9050 4200 9050
+Wire Wire Line
+	4200 9050 4550 9050
+Wire Wire Line
+	4550 9050 4900 9050
+Wire Wire Line
+	4900 9050 5250 9050
 Wire Wire Line
 	4900 9050 4900 9150
@@
 	3150 9450 3150 9550
 Wire Wire Line
-	3150 9550 5250 9550
+	3150 9550 3500 9550
+Wire Wire Line
+	3500 9550 3850 9550
+Wire Wire Line
+	3850 9550 4050 9550
+Wire Wire Line
+	4050 9550 4200 9550
+Wire Wire Line
+	4200 9550 4550 9550
+Wire Wire Line
+	4550 9550 4900 9550
+Wire Wire Line
+	4900 9550 5250 9550
 Wire Wire Line
 	4900 9550 4900 9450
@@
 	1850 6600 1950 6600
 Wire Wire Line
-	1850 2800 1850 7600
+	1850 2800 1850 3100
+Wire Wire Line
+	1850 3100 1850 3600
+Wire Wire Line
+	1850 3600 1850 4100
+Wire Wire Line
+	1850 4100 1850 4600
+Wire Wire Line
+	1850 4600 1850 5100
+Wire Wire Line
+	1850 5100 1850 5600
+Wire Wire Line
+	1850 5600 1850 6100
+Wire Wire Line
+	1850 6100 1850 6600
+Wire Wire Line
+	1850 6600 1850 7100
+Wire Wire Line
+	1850 7100 1850 7600
 Wire Wire Line
 	1850 3100 1950 3100
@@
 	1700 6700 1950 6700
 Wire Wire Line
-	1700 3200 1700 8200
+	1700 3200 1700 3700
+Wire Wire Line
+	1700 3700 1700 4200
+Wire Wire Line
+	1700 4200 1700 4700
+Wire Wire Line
+	1700 4700 1700 5200
+Wire Wire Line
+	1700 5200 1700 5700
+Wire Wire Line
+	1700 5700 1700 6200
+Wire Wire Line
+	1700 6200 1700 6700
+Wire Wire Line
+	1700 6700 1700 7200
+Wire Wire Line
+	1700 7200 1700 7700
+Wire Wire Line
+	1700 7700 1700 8200
 Wire Wire Line
 	1950 3200 1700 3200
@@
 	15050 8450 15050 8500
 Wire Wire Line
-	14500 8500 15250 8500
-Wire Wire Line
-	15150 8450 15150 8600
+	14500 8500 15050 8500
+Wire Wire Line
+	15050 8500 15150 8500
+Wire Wire Line
+	15150 8500 15250 8500
+Wire Wire Line
+	15150 8450 15150 8500
+Wire Wire Line
+	15150 8500 15150 8600
 Wire Wire Line
 	15250 8500 15250 8450
 Connection ~ 15150 8500
 Wire Wire Line
-	15150 6850 15150 7250
-Wire Wire Line
-	14500 7350 14500 8500
+	15150 6850 15150 6950
+Wire Wire Line
+	15150 6950 15150 7250
+Wire Wire Line
+	14500 7300 14500 8500
 Connection ~ 15050 8500
 Wire Wire Line
@@
 	10050 3350 9350 3350
 Wire Wire Line
-	11850 7200 11850 7300
+	11850 7200 11850 7250
+Wire Wire Line
+	11850 7250 11850 7300
 Wire Wire Line
 	12050 7200 12050 7300
@@
 	13650 2300 12950 2300
 Wire Wire Line
-	13350 5150 13800 5150
+	13350 5150 13700 5150
+Wire Wire Line
+	13700 5150 13800 5150
 Wire Wire Line
 	13700 5150 13700 4500
@@
 	9800 7950 9800 7900
 Wire Wire Line
-	9800 7450 9800 7600
+	9800 7450 9800 7550
+Wire Wire Line
+	9800 7550 9800 7600
 Wire Wire Line
 	9800 7550 9250 7550
@@
 	7400 5200 8300 5200
 Wire Wire Line
-	8300 5600 8300 5700
+	8300 5600 8300 5650
+Wire Wire Line
+	8300 5650 8300 5700
 Connection ~ 8300 5650
 Wire Wire Line
@@
 $EndComp
 Wire Wire Line
-	14250 7450 14600 7450
-Wire Wire Line
-	14400 7450 14400 7350
-$Comp
-L Conn_01x01 J?
+	14250 7450 14400 7450
+Wire Wire Line
+	14400 7450 14600 7450
+Wire Wire Line
+	14400 7450 14400 7300
+$Comp
+L Conn_01x01 J14
 U 1 1 5A6DCFAB
 P 14050 7450
-F 0 "J?" H 14050 7550 50  0000 C CNN
+F 0 "J14" H 14050 7550 50  0000 C CNN
 F 1 "Conn_01x01" H 14050 7350 50  0000 C CNN
-F 2 "" H 14050 7450 50  0001 C CNN
+F 2 "Pin_Headers:Pin_Header_Straight_1x01_Pitch2.54mm" H 14050 7450 50  0001 C CNN
 F 3 "" H 14050 7450 50  0001 C CNN
 	1    14050 7450
