File: Draco.sch (KiCad schematic (older format))
At the start: 32 parts, among them J1 Conn_01x03, J10 Conn_01x03, J11 Conn_01x06, J12 Conn_01x01, J13 Conn_02x05_Odd_Even, J2 Conn_01x03, J3 Conn_01x03, J4 Conn_01x03, J5 Conn_01x03, J6 Conn_01x03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

Commit message: replaced the level-shifter
Parts:
- removed U?: TXB0104D, Housings_SOIC:SOIC-14_3.9x8.7mm_Pitch1.27mm, symbol TXB0104D
- added U?: TXB0108DQSR, TO_SOT_Packages_SMD:USON-20_2x4mm_Pitch0.4mm, symbol TXB0108DQSR
Connections:
- net labels added: 5V_SCL, 5V_SDA
- wire segments 155 -> 205
Changed lines of the file:
@@
 GPS_RXD
 Text Label 8050 5000 2    60   ~ 0
-SDA
+5V_SDA
 Text Label 8050 4900 2    60   ~ 0
-SCL
+5V_SCL
 $Comp
 L RFM95HW U2
@@
 $EndComp
 Wire Wire Line
-	6350 7700 6350 7900
-Wire Wire Line
-	5950 7800 6350 7800
+	6350 7700 6350 7800
+Wire Wire Line
+	6350 7800 6350 7900
+Wire Wire Line
+	5950 7800 6050 7800
+Wire Wire Line
+	6050 7800 6150 7800
+Wire Wire Line
+	6150 7800 6250 7800
+Wire Wire Line
+	6250 7800 6350 7800
 Wire Wire Line
 	6250 7800 6250 7700
@@
 Connection ~ 6350 7800
 Wire Wire Line
-	5750 1700 5750 1900
-Wire Wire Line
-	5750 1800 6050 1800
+	5750 1700 5750 1800
+Wire Wire Line
+	5750 1800 5750 1900
+Wire Wire Line
+	5750 1800 5850 1800
+Wire Wire Line
+	5850 1800 5950 1800
+Wire Wire Line
+	5950 1800 6050 1800
 Wire Wire Line
 	6050 1800 6050 1900
@@
 Connection ~ 5750 1800
 Wire Wire Line
-	6250 1650 6250 1900
+	6250 1650 6250 1750
+Wire Wire Line
+	6250 1750 6250 1900
 Wire Wire Line
 	6250 1350 6250 1250
@@
 	6700 1750 6700 1850
 Wire Wire Line
-	4250 2500 4800 2500
-Wire Wire Line
-	4250 2800 4800 2800
+	4250 2500 4550 2500
+Wire Wire Line
+	4550 2500 4800 2500
+Wire Wire Line
+	4250 2800 4550 2800
+Wire Wire Line
+	4550 2800 4800 2800
 Connection ~ 4550 2500
 Connection ~ 4550 2800
@@
 	3950 2500 3800 2500
 Wire Wire Line
-	3800 2500 3800 2850
+	3800 2500 3800 2800
+Wire Wire Line
+	3800 2800 3800 2850
 Wire Wire Line
 	3800 2800 3950 2800
 Connection ~ 3800 2800
 Wire Wire Line
-	3800 2200 4800 2200
+	3800 2200 4350 2200
+Wire Wire Line
+	4350 2200 4650 2200
+Wire Wire Line
+	4650 2200 4800 2200
 Wire Wire Line
 	4650 2200 4650 2100
@@
 	10050 9150 10250 9150
 Wire Wire Line
-	10250 9150 10250 9650
+	10250 9150 10250 9250
+Wire Wire Line
+	10250 9250 10250 9350
+Wire Wire Line
+	10250 9350 10250 9450
+Wire Wire Line
+	10250 9450 10250 9650
 Wire Wire Line
 	10050 9450 10250 9450
@@
 	3150 9150 3150 9050
 Wire Wire Line
-	3150 9050 5250 9050
+	3150 9050 3500 9050
+Wire Wire Line
+	3500 9050 3850 9050
+Wire Wire Line
+	3850 9050 4050 9050
+Wire Wire Line
+	4050 9050 4200 9050
+Wire Wire Line
+	4200 9050 4550 9050
+Wire Wire Line
+	4550 9050 4900 9050
+Wire Wire Line
+	4900 9050 5250 9050
 Wire Wire Line
 	4900 9050 4900 9150
@@
 	3150 9450 3150 9550
 Wire Wire Line
-	3150 9550 5250 9550
+	3150 9550 3500 9550
+Wire Wire Line
+	3500 9550 3850 9550
+Wire Wire Line
+	3850 9550 4050 9550
+Wire Wire Line
+	4050 9550 4200 9550
+Wire Wire Line
+	4200 9550 4550 9550
+Wire Wire Line
+	4550 9550 4900 9550
+Wire Wire Line
+	4900 9550 5250 9550
 Wire Wire Line
 	4900 9550 4900 9450
@@
 	1850 6600 1950 6600
 Wire Wire Line
-	1850 2700 1850 7600
+	1850 2700 1850 3100
+Wire Wire Line
+	1850 3100 1850 3600
+Wire Wire Line
+	1850 3600 1850 4100
+Wire Wire Line
+	1850 4100 1850 4600
+Wire Wire Line
+	1850 4600 1850 5100
+Wire Wire Line
+	1850 5100 1850 5600
+Wire Wire Line
+	1850 5600 1850 6100
+Wire Wire Line
+	1850 6100 1850 6600
+Wire Wire Line
+	1850 6600 1850 7100
+Wire Wire Line
+	1850 7100 1850 7600
 Wire Wire Line
 	1850 3100 1950 3100
@@
 	1700 6700 1950 6700
 Wire Wire Line
-	1700 3200 1700 8200
+	1700 3200 1700 3700
+Wire Wire Line
+	1700 3700 1700 4200
+Wire Wire Line
+	1700 4200 1700 4700
+Wire Wire Line
+	1700 4700 1700 5200
+Wire Wire Line
+	1700 5200 1700 5700
+Wire Wire Line
+	1700 5700 1700 6200
+Wire Wire Line
+	1700 6200 1700 6700
+Wire Wire Line
+	1700 6700 1700 7200
+Wire Wire Line
+	1700 7200 1700 7700
+Wire Wire Line
+	1700 7700 1700 8200
 Wire Wire Line
 	1950 3200 1700 3200
@@
 	15400 8500 15400 8550
 Wire Wire Line
-	14850 8550 15600 8550
-Wire Wire Line
-	15500 8500 15500 8650
+	14850 8550 15400 8550
+Wire Wire Line
+	15400 8550 15500 8550
+Wire Wire Line
+	15500 8550 15600 8550
+Wire Wire Line
+	15500 8500 15500 8550
+Wire Wire Line
+	15500 8550 15500 8650
 Wire Wire Line
 	15600 8550 15600 8500
@@
 	14050 8000 14950 8000
 Wire Wire Line
-	14650 7500 14950 7500
+	14650 7500 14750 7500
+Wire Wire Line
+	14750 7500 14950 7500
 Wire Wire Line
 	14750 7500 14750 7400
 Connection ~ 14750 7500
-$Comp
-L TXB0104D U?
-U 1 1 5A5C5F5D
-P 13250 7900
-F 0 "U?" H 12975 8555 50  0000 C CNN
-F 1 "TXB0104D" H 13600 8550 50  0000 C CNN
-F 2 "Housings_SOIC:SOIC-14_3.9x8.7mm_Pitch1.27mm" H 13300 7050 50  0001 C CNN
-F 3 "" H 13360 7995 50  0001 C CNN
-	1    13250 7900
-	-1   0    0    -1
-$EndComp
 Wire Wire Line
 	13950 7700 13950 7600
@@
 	14050 8200 14050 8000
 Wire Wire Line
-	13350 7200 13350 7100
-Wire Wire Line
-	13150 7200 13150 7100
-Wire Wire Line
-	13250 8600 13250 8700
+	9350 4350 9350 4250
+Wire Wire Line
+	9550 4350 9550 4250
+Wire Wire Line
+	9450 5750 9450 5850
 $Comp
 L GND #PWR019
 U 1 1 5A5C6BD9
-P 13250 8700
-F 0 "#PWR019" H 13250 8450 50  0001 C CNN
-F 1 "GND" H 13250 8550 50  0000 C CNN
-F 2 "" H 13250 8700 50  0001 C CNN
-F 3 "" H 13250 8700 50  0001 C CNN
-	1    13250 8700
+P 9450 5850
+F 0 "#PWR019" H 9450 5600 50  0001 C CNN
+F 1 "GND" H 9450 5700 50  0000 C CNN
+F 2 "" H 9450 5850 50  0001 C CNN
+F 3 "" H 9450 5850 50  0001 C CNN
+	1    9450 5850
 	1    0    0    -1
 $EndComp
@@
 L +3.3V #PWR020
 U 1 1 5A5C6C80
-P 13350 7100
-F 0 "#PWR020" H 13350 6950 50  0001 C CNN
-F 1 "+3.3V" H 13350 7240 50  0000 C CNN
-F 2 "" H 13350 7100 50  0001 C CNN
-F 3 "" H 13350 7100 50  0001 C CNN
-	1    13350 7100
+P 9350 4250
+F 0 "#PWR020" H 9350 4100 50  0001 C CNN
+F 1 "+3.3V" H 9350 4390 50  0000 C CNN
+F 2 "" H 9350 4250 50  0001 C CNN
+F 3 "" H 9350 4250 50  0001 C CNN
+	1    9350 4250
 	1    0    0    -1
 $EndComp
@@
 L +5V #PWR021
 U 1 1 5A5C6D09
-P 13150 7100
-F 0 "#PWR021" H 13150 6950 50  0001 C CNN
-F 1 "+5V" H 13150 7240 50  0000 C CNN
-F 2 "" H 13150 7100 50  0001 C CNN
-F 3 "" H 13150 7100 50  0001 C CNN
-	1    13150 7100
-	1    0    0    -1
-$EndComp
-Wire Wire Line
-	12850 7800 12350 7800
-Wire Wire Line
-	12850 7600 12350 7600
-Wire Wire Line
-	12850 8000 12350 8000
-Wire Wire Line
-	12850 8200 12350 8200
-Text Label 12350 7600 0    60   ~ 0
+P 9550 4250
+F 0 "#PWR021" H 9550 4100 50  0001 C CNN
+F 1 "+5V" H 9550 4390 50  0000 C CNN
+F 2 "" H 9550 4250 50  0001 C CNN
+F 3 "" H 9550 4250 50  0001 C CNN
+	1    9550 4250
+	1    0    0    -1
+$EndComp
+Wire Wire Line
+	13400 7800 12900 7800
+Wire Wire Line
+	13400 7600 12900 7600
+Wire Wire Line
+	13400 8000 12900 8000
+Wire Wire Line
+	13400 8200 12900 8200
+Text Label 12900 7600 0    60   ~ 0
 LORA_NSS
-Text Label 12350 7800 0    60   ~ 0
+Text Label 12900 7800 0    60   ~ 0
 MOSI
-Text Label 12350 8000 0    60   ~ 0
+Text Label 12900 8000 0    60   ~ 0
 MISO
-Text Label 12350 8200 0    60   ~ 0
+Text Label 12900 8200 0    60   ~ 0
 SCK
 Wire Wire Line
@@
 F1 "imu.sch" 60
 $EndSheet
+$Comp
+L TXB0108DQSR U?
+U 1 1 5A5FEA4F
+P 9450 5050
+F 0 "U?" H 9800 5700 50  0000 L CNN
+F 1 "TXB0108DQSR" H 9800 5600 50  0000 L CNN
+F 2 "TO_SOT_Packages_SMD:USON-20_2x4mm_Pitch0.4mm" H 9800 5500 50  0001 L CNN
+F 3 "" H 9450 4950 50  0001 C CNN
+	1    9450 5050
+	1    0    0    -1
+$EndComp
 $EndSCHEMATC

Commit message: added sd card
Parts:
- removed U?: TXB0108DQSR, TO_SOT_Packages_SMD:USON-20_2x4mm_Pitch0.4mm, symbol TXB0108DQSR
- added C?: 100nF, symbol C
- added J17: Micro_SD_Card, symbol Micro_SD_Card
- added Q?: 2N3904, TO_SOT_Packages_THT:TO-92_Molded_Narrow, symbol 2N3904
- added R? (x2): 1k, symbol R
- added U6: LOGIC-TXS0108EPWR(TSSOP20), TSSOP20-0.65-6.5X4.4MM, symbol LOGIC-TXS0108EPWR(TSSOP20)
Connections:
- net labels added: 3V_LORA_NSS, 3V_LORA_RST, 3V_MISO, 3V_MOSI, 3V_SCK, 3V_SCL, 3V_SDA, 3V_SD_NSS, 5V_LORA_NSS, 5V_LORA_RST, 5V_MISO, 5V_MOSI, 5V_SCK, 5V_SD_NSS, LORA_INT, PROG_RX, PROG_TX
- net labels removed: LORA_NSS, MISO, MOSI, RX, SCK, SCL, SDA, TX
- wire segments 205 -> 194
Other:
- note added: "//TODO Figure out the reset on the LORA module"
- note added: "//TODO Leave pins floating?"
- moved on the sheet: AE1, J12, L1, U2

Commit message: Did design review. Changed/confirmed voltage levels
Parts:
- removed Q?: 2N3904, TO_SOT_Packages_THT:TO-92_Molded_Narrow, symbol 2N3904
- removed R? (x2): 1k, symbol R
- added C13: 100nF, Capacitors_SMD:C_0805, symbol C
- added D1, D2, D3: LED, LEDs:LED_0805, symbol LED
- added J13: Conn_01x04, symbol Conn_01x04
- added JP1: Jumper_NC_Dual, symbol Jumper_NC_Dual
- added R10: 4.7K, Resistors_SMD:R_0805, symbol R
- added R11, R9: 0, Resistors_SMD:R_0805, symbol R
- added R2, R3, R4, R7, R8: 1k, Resistors_SMD:R_0805, symbol R
- added R5: 20k, Resistors_SMD:R_0805, symbol R
- added R6: 10k, Resistors_SMD:R_0805, symbol R
- C1: renamed from C6; footprint (none) -> Capacitors_SMD:C_0805
- C10: renamed from C11; footprint (none) -> Capacitors_SMD:C_0805
- C12: renamed from C5; footprint (none) -> Capacitors_SMD:C_0805
- C14: renamed from C?; footprint (none) -> Capacitors_SMD:C_0805
- C2: renamed from C7; footprint (none) -> Capacitors_SMD:C_0805
- C3: renamed from C8; footprint (none) -> Capacitors_SMD:C_0805
- C4: renamed from C1; footprint (none) -> Capacitors_SMD:C_0805
- C5: renamed from C2; footprint (none) -> Capacitors_SMD:C_0805
- C6: renamed from C9; footprint (none) -> Capacitors_SMD:C_0805
- C7: renamed from C3; footprint (none) -> Capacitors_SMD:C_0805
- C8: renamed from C10; footprint (none) -> Capacitors_SMD:C_0805
- R1: footprint (none) -> Resistors_SMD:R_0805
- U1: footprint TQFP100 -> Housings_QFP:TQFP-100_14x14mm_Pitch0.5mm
- U2: renamed from U6; footprint TSSOP20-0.65-6.5X4.4MM -> SMD_Packages:SSOP-20
- U3: renamed from U2; footprint mysensors_radios:RFM69HW_SMD_ThroughHole_Handsoldering -> (none)
- renumbered C12 to C11, C4 to C9, J13 to J12, J12 to J14, J17 to J15
Connections:
- net +3V3: now also C13.1
- net +5V: now also JP1.3
- net +BATT: now also R5.2; no longer J1.2 (Pin_2), J10.2 (Pin_2), J2.2 (Pin_2), J3.2 (Pin_2), J4.2 (Pin_2), J5.2 (Pin_2), J6.2 (Pin_2), J7.2 (Pin_2), J8.2 (Pin_2), J9.2 (Pin_2)
- net 3V_LORA_RST: now also U2.9 (A8); no longer U2.12 (B8)
- net 3V_SD_NSS: no longer U2.13 (B7)
- net 5V_LORA_RST: now also U1.93 ((TCK/ADC4)PF4), U2.12 (B8); no longer U2.9 (A8)
- net 5V_SD_NSS: now also U2.13 (B7)
- net GND: now also C13.2, D1.1 (K), D2.1 (K), D3.1 (K), J13.4 (Pin_4), R3.1, R6.1
- net GPS_RXD: now also R2.1, R3.2; no longer U1.46 ((TXD1/INT3)PD3)
- net LORA_INT: now also U1.6 ((OC3B/INT4)PE4)
- net SERVO10: now also U1.8 ((T3/INT6)PE6); no longer U1.28 (PG3(TOSC2))
- net SERVO9: now also U1.9 ((CLKO/ICP3/INT7)PE7); no longer U1.27 (PH7(T4))
- net LED_RED: now reaches U1.15 (PH3(OC4A))
- net LED_RED: now also R4.2
- net LED_YELLOW: now reaches U1.16 (PH4(OC4B))
- net LED_YELLOW: now also R7.2
- net LED_GREEN: now reaches U1.17 (PH5(OC4C))
- net LED_GREEN: now also R8.2
- net CAM_LED: now reaches U1.66 (PJ3(PCINT12))
- net CAM_LED: now also R9.2
- net CAM_PHOTO: now reaches U1.67 (PJ4(PCINT13))
- net CAM_PHOTO: now also R11.2
- net CAM_PWR: now reaches U1.68 (PJ5(PCINT14))
- net CAM_PWR: now also R10.2
- net GPS_INT: now reaches U1.7 ((OC3C/INT5)PE5)
- net GYRO_INT1: now reaches U1.85 (PK4(ADC12/PCINT20))
- net GYRO_INT2: now reaches U1.86 (PK3(ADC11/PCINT19))
- net ACCEL_INT1: now reaches U1.87 (PK2(ADC10/PCINT18))
- net ACCEL_INT2: now reaches U1.88 (PK1(ADC9/PCINT17))
- net MAGNET_INT1: now reaches U1.89 (PK0(ADC8/PCINT16))
- net VBAT: now reaches U1.94 ((ADC3)PF3)
- net VBAT: now also R5.1, R6.2
- new net: R2.2, U1.46 ((TXD1/INT3)PD3)
- new net: J1.2 (Pin_2), J10.2 (Pin_2), J2.2 (Pin_2), J3.2 (Pin_2), J4.2 (Pin_2), J5.2 (Pin_2), J6.2 (Pin_2), J7.2 (Pin_2), J8.2 (Pin_2), J9.2 (Pin_2), JP1.2
- new net: J13.1 (Pin_1), R9.1
- new net: J13.2 (Pin_2), R10.1
- new net: J13.3 (Pin_3), R11.1
- new net: D1.2 (A), R4.1
- new net: D2.2 (A), R7.1
- new net: D3.2 (A), R8.1
- new net VCC: JP1.1
Other:
- note added: "//5V AVR should have a 3.0V threshold for interrupts"
- note added: "//Choose between HV servos and 5V"
- note added: "5mA through each LED\n"
- note added: "CAM_PWR needs 9.8k-3.13k"
- note removed: "//TODO Figure out the reset on the LORA module"
- note removed: "//TODO Leave pins floating?"
- moved on the sheet: J15

Commit message: Started Board layout
Parts:
- AE1: footprint (none) -> Current_Control_Systems:U.FL-R-SMT
- C11, C9: footprint (none) -> Capacitors_THT:CP_Radial_D5.0mm_P2.00mm
- J1, J10, J2, J3, J4, J5, J6, J7, J8, J9, JP1: footprint (none) -> Pin_Headers:Pin_Header_Straight_1x03_Pitch2.54mm
- J11: footprint (none) -> Connectors_JST:JST_PH_B6B-PH-K_06x2.00mm_Straight
- J12: footprint (none) -> Pin_Headers:Pin_Header_Straight_2x05_Pitch2.54mm
- J13: footprint (none) -> Connectors_JST:JST_PH_B4B-PH-K_04x2.00mm_Straight
- J14: footprint (none) -> Pin_Headers:Pin_Header_Straight_1x01_Pitch2.54mm
- J15: footprint (none) -> Connectors:microSD_Card_Receptacle_Wuerth_693072010801
- L1: footprint (none) -> Inductors_SMD:L_0805
- U3: footprint (none) -> RF_Modules:Hopref_RFM9XW_SMD
- Y1: footprint (none) -> Crystals:Crystal_SMD_HC49-SD
Connections:
- net 5V_LORA_RST: now also U1.92 ((TMS/ADC5)PF5); no longer U1.93 ((TCK/ADC4)PF4)
- new net VBAT2: U1.93 ((TCK/ADC4)PF4)
Changed lines of the file:
@@
 LIBS:TXB0104DR
 LIBS:LOGIC-TXS0108EPWR_TSSOP20_
+LIBS:CurrentControlSystems
 LIBS:Draco-cache
 EELAYER 25 0
@@
 $EndDescr
 $Sheet
-S 14950 1950 750  1500
+S 15300 1950 750  1500
 U 5A59AC7F
 F0 "Power Supply" 60
 F1 "power.sch" 60
+F2 "VBAT2" O L 15300 2150 60
 $EndSheet
 $Comp
@@
 F 0 "L1" V 6200 1450 50  0000 C CNN
 F 1 "10uH" V 6325 1450 50  0000 C CNN
-F 2 "" H 6250 1450 50  0001 C CNN
+F 2 "Inductors_SMD:L_0805" H 6250 1450 50  0001 C CNN
 F 3 "" H 6250 1450 50  0001 C CNN
 	1    6250 1450
@@
 F 0 "Y1" H 4550 2800 50  0000 C CNN
 F 1 "16MHz" H 4550 2500 50  0000 C CNN
-F 2 "" H 4550 2650 50  0001 C CNN
+F 2 "Crystals:Crystal_SMD_HC49-SD" H 4550 2650 50  0001 C CNN
 F 3 "" H 4550 2650 50  0001 C CNN
 	1    4550 2650
@@
 F 0 "J12" H 9800 9550 50  0000 C CNN
 F 1 "Conn_02x05_Odd_Even" H 9800 8950 50  0000 C CNN
-F 2 "" H 9750 9250 50  0001 C CNN
+F 2 "Pin_Headers:Pin_Header_Straight_2x05_Pitch2.54mm" H 9750 9250 50  0001 C CNN
 F 3 "" H 9750 9250 50  0001 C CNN
 	1    9750 9250
@@
 F 0 "C9" H 4725 7700 50  0000 L CNN
 F 1 "0.1uF" H 4725 7500 50  0000 L CNN
-F 2 "" H 4738 7450 50  0001 C CNN
+F 2 "Capacitors_THT:CP_Radial_D5.0mm_P2.00mm" H 4738 7450 50  0001 C CNN
 F 3 "" H 4700 7600 50  0001 C CNN
 	1    4700 7600
@@
 F 0 "J11" H 7800 9450 50  0000 C CNN
 F 1 "Conn_01x06" H 7800 8750 50  0000 C CNN
-F 2 "" H 7800 9150 50  0001 C CNN
+F 2 "Connectors_JST:JST_PH_B6B-PH-K_06x2.00mm_Straight" H 7800 9150 50  0001 C CNN
 F 3 "" H 7800 9150 50  0001 C CNN
 	1    7800 9150
@@
 F 0 "J1" H 2150 3300 50  0000 C CNN
 F 1 "Conn_01x03" H 2150 2900 50  0000 C CNN
-F 2 "" H 2150 3100 50  0001 C CNN
+F 2 "Pin_Headers:Pin_Header_Straight_1x03_Pitch2.54mm" H 2150 3100 50  0001 C CNN
 F 3 "" H 2150 3100 50  0001 C CNN
 	1    2150 3100
@@
 F 0 "J2" H 2150 3800 50  0000 C CNN
 F 1 "Conn_01x03" H 2150 3400 50  0000 C CNN
-F 2 "" H 2150 3600 50  0001 C CNN
+F 2 "Pin_Headers:Pin_Header_Straight_1x03_Pitch2.54mm" H 2150 3600 50  0001 C CNN
 F 3 "" H 2150 3600 50  0001 C CNN
 	1    2150 3600
@@
 F 0 "J3" H 2150 4300 50  0000 C CNN
 F 1 "Conn_01x03" H 2150 3900 50  0000 C CNN
-F 2 "" H 2150 4100 50  0001 C CNN
+F 2 "Pin_Headers:Pin_Header_Straight_1x03_Pitch2.54mm" H 2150 4100 50  0001 C CNN
 F 3 "" H 2150 4100 50  0001 C CNN
 	1    2150 4100
@@
 F 0 "J4" H 2150 4800 50  0000 C CNN
 F 1 "Conn_01x03" H 2150 4400 50  0000 C CNN
-F 2 "" H 2150 4600 50  0001 C CNN
+F 2 "Pin_Headers:Pin_Header_Straight_1x03_Pitch2.54mm" H 2150 4600 50  0001 C CNN
 F 3 "" H 2150 4600 50  0001 C CNN
 	1    2150 4600
@@
 F 0 "J5" H 2150 5300 50  0000 C CNN
 F 1 "Conn_01x03" H 2150 4900 50  0000 C CNN
-F 2 "" H 2150 5100 50  0001 C CNN
+F 2 "Pin_Headers:Pin_Header_Straight_1x03_Pitch2.54mm" H 2150 5100 50  0001 C CNN
 F 3 "" H 2150 5100 50  0001 C CNN
 	1    2150 5100
@@
 F 0 "J6" H 2150 5800 50  0000 C CNN
 F 1 "Conn_01x03" H 2150 5400 50  0000 C CNN
-F 2 "" H 2150 5600 50  0001 C CNN
+F 2 "Pin_Headers:Pin_Header_Straight_1x03_Pitch2.54mm" H 2150 5600 50  0001 C CNN
 F 3 "" H 2150 5600 50  0001 C CNN
 	1    2150 5600
@@
 F 0 "J7" H 2150 6300 50  0000 C CNN
 F 1 "Conn_01x03" H 2150 5900 50  0000 C CNN
-F 2 "" H 2150 6100 50  0001 C CNN
+F 2 "Pin_Headers:Pin_Header_Straight_1x03_Pitch2.54mm" H 2150 6100 50  0001 C CNN
 F 3 "" H 2150 6100 50  0001 C CNN
 	1    2150 6100
@@
 F 0 "J8" H 2150 6800 50  0000 C CNN
 F 1 "Conn_01x03" H 2150 6400 50  0000 C CNN
-F 2 "" H 2150 6600 50  0001 C CNN
+F 2 "Pin_Headers:Pin_Header_Straight_1x03_Pitch2.54mm" H 2150 6600 50  0001 C CNN
 F 3 "" H 2150 6600 50  0001 C CNN
 	1    2150 6600
@@
 F 0 "J9" H 2150 7300 50  0000 C CNN
 F 1 "Conn_01x03" H 2150 6900 50  0000 C CNN
-F 2 "" H 2150 7100 50  0001 C CNN
+F 2 "Pin_Headers:Pin_Header_Straight_1x03_Pitch2.54mm" H 2150 7100 50  0001 C CNN
 F 3 "" H 2150 7100 50  0001 C CNN
 	1    2150 7100
@@
 F 0 "J10" H 2150 7800 50  0000 C CNN
 F 1 "Conn_01x03" H 2150 7400 50  0000 C CNN
-F 2 "" H 2150 7600 50  0001 C CNN
+F 2 "Pin_Headers:Pin_Header_Straight_1x03_Pitch2.54mm" H 2150 7600 50  0001 C CNN
 F 3 "" H 2150 7600 50  0001 C CNN
 	1    2150 7600
@@
 F 0 "C11" H 5275 9400 50  0000 L CNN
 F 1 "10uF" H 5275 9200 50  0000 L CNN
-F 2 "" H 5288 9150 50  0001 C CNN
+F 2 "Capacitors_THT:CP_Radial_D5.0mm_P2.00mm" H 5288 9150 50  0001 C CNN
 F 3 "" H 5250 9300 50  0001 C CNN
 	1    5250 9300
@@
 F 0 "U3" H 14800 7850 40  0000 C CNN
 F 1 "RFM95HW" H 15400 6850 40  0000 C CNN
-F 2 "" H 15150 7600 30  0001 C CIN
+F 2 "RF_Modules:Hopref_RFM9XW_SMD" H 15150 7600 30  0001 C CIN
 F 3 "" H 15150 7600 60  0000 C CNN
 	1    15150 7600
@@
 F 0 "AE1" H 14325 7325 50  0000 R CNN
 F 1 "Antenna_Shield" H 14325 7250 50  0000 R CNN
-F 2 "" H 14400 7250 50  0001 C CNN
+F 2 "Current_Control_Systems:U.FL-R-SMT" H 14400 7250 50  0001 C CNN
 F 3 "" H 14400 7250 50  0001 C CNN
 	1    14400 7150
@@
 F 0 "J14" H 14100 7550 50  0000 C CNN
 F 1 "Conn_01x01" H 14100 7350 50  0000 C CNN
-F 2 "" H 14100 7450 50  0001 C CNN
+F 2 "Pin_Headers:Pin_Header_Straight_1x01_Pitch2.54mm" H 14100 7450 50  0001 C CNN
 F 3 "" H 14100 7450 50  0001 C CNN
 	1    14100 7450
@@
 F 0 "J15" H 14050 5750 50  0000 C CNN
 F 1 "Micro_SD_Card" H 15350 5750 50  0000 R CNN
-F 2 "" H 15850 5450 50  0001 C CNN
+F 2 "Connectors:microSD_Card_Receptacle_Wuerth_693072010801" H 15850 5450 50  0001 C CNN
 F 3 "" H 14700 5150 50  0001 C CNN
 	1    14700 5150
@@
 F 0 "JP1" H 1900 2600 50  0000 L CNN
 F 1 "Jumper_NC_Dual" H 1850 2800 50  0000 C BNN
-F 2 "" H 1850 2700 50  0001 C CNN
+F 2 "Pin_Headers:Pin_Header_Straight_1x03_Pitch2.54mm" H 1850 2700 50  0001 C CNN
 F 3 "" H 1850 2700 50  0001 C CNN
 	1    1850 2700
@@
 F 0 "J13" H 12150 5300 50  0000 C CNN
 F 1 "Conn_01x04" H 12150 4800 50  0000 C CNN
-F 2 "" H 12150 5100 50  0001 C CNN
+F 2 "Connectors_JST:JST_PH_B4B-PH-K_04x2.00mm_Straight" H 12150 5100 50  0001 C CNN
 F 3 "" H 12150 5100 50  0001 C CNN
 	1    12150 5100
@@
 VBAT
 Wire Wire Line
-	7400 7100 8050 7100
-Text Label 8050 7100 2    60   ~ 0
+	7400 7200 8050 7200
+Text Label 8050 7200 2    60   ~ 0
 5V_LORA_RST
 $Comp
@@
 Wire Wire Line
 	8300 5200 8300 5300
+Wire Wire Line
+	15300 2150 14850 2150
+Text Label 14850 2150 0    60   ~ 0
+VBAT2
+Wire Wire Line
+	7400 7100 8050 7100
+Text Label 8050 7100 2    60   ~ 0
+VBAT2
 $EndSCHEMATC

Commit message: pushed new psu to pcb
Parts:
- C11, C9: footprint Capacitors_THT:CP_Radial_D5.0mm_P2.00mm -> Capacitors_SMD:C_0805
Changed lines of the file:
@@
 F 0 "C9" H 4725 7700 50  0000 L CNN
 F 1 "0.1uF" H 4725 7500 50  0000 L CNN
-F 2 "Capacitors_THT:CP_Radial_D5.0mm_P2.00mm" H 4738 7450 50  0001 C CNN
+F 2 "Capacitors_SMD:C_0805" H 4738 7450 50  0001 C CNN
 F 3 "" H 4700 7600 50  0001 C CNN
 	1    4700 7600
@@
 F 0 "C11" H 5275 9400 50  0000 L CNN
 F 1 "10uF" H 5275 9200 50  0000 L CNN
-F 2 "Capacitors_THT:CP_Radial_D5.0mm_P2.00mm" H 5288 9150 50  0001 C CNN
+F 2 "Capacitors_SMD:C_0805" H 5288 9150 50  0001 C CNN
 F 3 "" H 5250 9300 50  0001 C CNN
 	1    5250 9300
