File: Draco.sch (KiCad schematic (older format))
At the start: 51 parts, among them J1 Conn_01x03, J10 Conn_01x03, J11 Conn_01x06, J12 Conn_02x05_Odd_Even, J13 Conn_01x04, J15 Micro_SD_Card, J2 Conn_01x03, J20 Conn_01x04, J3 Conn_01x03, J4 Conn_01x03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

Commit message: Adding bypass capacitors
Parts:
- J14: renamed from J?; footprint (none) -> Pin_Headers:Pin_Header_Straight_1x01_Pitch2.54mm
Connections:
- net ACCEL_INT1: now also U1.88 (PK1(ADC9/PCINT17)); no longer U1.87 (PK2(ADC10/PCINT18))
- net ACCEL_INT2: now also U1.87 (PK2(ADC10/PCINT18)); no longer U1.88 (PK1(ADC9/PCINT17))
- net GYRO_INT1: no longer names the net of U1.85 (PK4(ADC12/PCINT20))
- net GYRO_INT2: no longer names the net of U1.86 (PK3(ADC11/PCINT19))
Changed lines of the file:
@@
 F4 "ACCEL_INT1" O L 13650 2450 60
 F5 "ACCEL_INT2" O L 13650 2600 60
-F6 "GYRO_INT1" O L 13650 2750 60
-F7 "GYRO_INT2" O L 13650 2900 60
 F8 "MAGNET_INT1" O L 13650 3050 60
 $EndSheet
@@
 Text Label 12950 2600 0    60   ~ 0
 ACCEL_INT2
-Text Label 12950 2750 0    60   ~ 0
-GYRO_INT1
-Text Label 12950 2900 0    60   ~ 0
-GYRO_INT2
 Text Label 12950 3050 0    60   ~ 0
 MAGNET_INT1
+Text Label 4200 4100 0    60   ~ 0
+ACCEL_INT1
 Text Label 4200 4200 0    60   ~ 0
-ACCEL_INT1
-Text Label 4200 4100 0    60   ~ 0
 ACCEL_INT2
 Text Label 4200 4000 0    60   ~ 0
 MAGNET_INT1
-Text Label 4200 4400 0    60   ~ 0
-GYRO_INT1
-Text Label 4200 4300 0    60   ~ 0
-GYRO_INT2
 Text Label 11150 2850 0    60   ~ 0
 GPS_INT
@@
 	13650 2600 12950 2600
 Wire Wire Line
-	13650 2750 12950 2750
-Wire Wire Line
-	13650 2900 12950 2900
-Wire Wire Line
 	13650 3050 12950 3050
 Wire Wire Line
+	4800 4100 4200 4100
+Wire Wire Line
 	4800 4200 4200 4200
 Wire Wire Line
-	4800 4100 4200 4100
-Wire Wire Line
 	4800 4000 4200 4000
-Wire Wire Line
-	4800 4400 4200 4400
-Wire Wire Line
-	4800 4300 4200 4300
 Wire Wire Line
 	11700 2850 11150 2850
@@
 	14400 7450 14400 7350
 $Comp
-L Conn_01x01 J?
+L Conn_01x01 J14
 U 1 1 5A6DCFAB
 P 14050 7450
-F 0 "J?" H 14050 7550 50  0000 C CNN
+F 0 "J14" H 14050 7550 50  0000 C CNN
 F 1 "Conn_01x01" H 14050 7350 50  0000 C CNN
-F 2 "" H 14050 7450 50  0001 C CNN
+F 2 "Pin_Headers:Pin_Header_Straight_1x01_Pitch2.54mm" H 14050 7450 50  0001 C CNN
 F 3 "" H 14050 7450 50  0001 C CNN
 	1    14050 7450

Commit message: Added camera resistor divider
Parts:
- added R38, R39, R40: 0, Resistors_SMD:R_0805, symbol R
- R2: value 1k -> 2k7
- R3: value 1k -> 4k7
Connections:
- net GND: now also R38.1, R39.1, R40.1
- net SERVO10: now also U1.52 (PG1(~RD~)); no longer U1.8 ((T3/INT6)PE6)
- net SERVO9: now also U1.51 (PG0(~WR~)); no longer U1.9 ((CLKO/ICP3/INT7)PE7)
- net at J13.1 (Pin_1), R9.1: now also R40.2
- net at J13.2 (Pin_2), R10.1: now also R39.2
- net at J13.3 (Pin_3), R11.1: now also R38.2
- net ~FIRE_A renamed FIRE_A
- net ~FIRE_B renamed FIRE_B
- net ~FIRE_C renamed FIRE_C
Other:
- note removed: "//5V AVR should have a 3.0V threshold for interrupts"
- moved on the sheet: R10, R11, R9
Changed lines of the file:
@@
 F2 "TEST_EN_A" I L 10050 2150 60
 F3 "TEST_READ_A" O L 10050 2300 60
-F4 "~FIRE_A" I L 10050 2450 60
-F5 "TEST_EN_B" I L 10050 2600 60
-F6 "TEST_READ_B" O L 10050 2750 60
-F7 "~FIRE_B" I L 10050 2900 60
-F8 "TEST_EN_C" I L 10050 3050 60
-F9 "TEST_READ_C" O L 10050 3200 60
-F10 "~FIRE_C" I L 10050 3350 60
+F4 "TEST_EN_B" I L 10050 2600 60
+F5 "TEST_READ_B" O L 10050 2750 60
+F6 "TEST_EN_C" I L 10050 3050 60
+F7 "TEST_READ_C" O L 10050 3200 60
+F8 "FIRE_A" I L 10050 2450 60
+F9 "FIRE_B" I L 10050 2900 60
+F10 "FIRE_C" I L 10050 3350 60
 $EndSheet
 Text Label 9350 2150 0    60   ~ 0
@@
 TEST_READ_A
 Text Label 9350 2450 0    60   ~ 0
-~FIRE_A
+FIRE_A
 Text Label 9350 2600 0    60   ~ 0
 TEST_EN_B
@@
 TEST_READ_B
 Text Label 9350 2900 0    60   ~ 0
-~FIRE_B
+FIRE_B
 Text Label 8050 6700 2    60   ~ 0
 TEST_READ_A
@@
 TEST_READ_B
 Text Label 8050 2200 2    60   ~ 0
-~FIRE_A
+FIRE_A
 Text Label 8050 2300 2    60   ~ 0
-~FIRE_B
+FIRE_B
 Text Label 8050 2500 2    60   ~ 0
 TEST_EN_A
@@
 TEST_EN_C
 Text Label 8050 2400 2    60   ~ 0
-~FIRE_C
+FIRE_C
 Text Label 8050 6900 2    60   ~ 0
 TEST_READ_C
@@
 TEST_READ_C
 Text Label 9350 3350 0    60   ~ 0
-~FIRE_C
+FIRE_C
 $Sheet
 S 13650 1950 750  1500
@@
 F4 "ACCEL_INT1" O L 13650 2450 60
 F5 "ACCEL_INT2" O L 13650 2600 60
-F8 "MAGNET_INT1" O L 13650 3050 60
+F6 "MAGNET_INT1" O L 13650 3050 60
 $EndSheet
 $Comp
@@
 Text Label 4200 3800 0    60   ~ 0
 SERVO8
-Text Label 8050 6500 2    60   ~ 0
+Text Label 4200 6700 0    60   ~ 0
 SERVO9
-Text Label 8050 6400 2    60   ~ 0
+Text Label 4200 6800 0    60   ~ 0
 SERVO10
 Text Label 16200 7600 2    60   ~ 0
@@
 	1    0    0    -1
 $EndComp
-Text Notes 8150 6350 0    60   ~ 0
-//5V AVR should have a 3.0V threshold for interrupts
 Text Label 12950 2450 0    60   ~ 0
 ACCEL_INT1
@@
 	4800 3800 4200 3800
 Wire Wire Line
-	7400 6500 8050 6500
-Wire Wire Line
-	7400 6400 8050 6400
+	4800 6700 4200 6700
+Wire Wire Line
+	4800 6800 4200 6800
 Wire Wire Line
 	11500 7500 11400 7500
@@
 	1450 2700 1450 2550
 Wire Wire Line
-	11650 5000 11100 5000
-Wire Wire Line
-	11650 5200 11100 5200
-Wire Wire Line
-	11650 5100 11100 5100
+	11150 5000 10600 5000
+Wire Wire Line
+	11150 5200 10600 5200
+Wire Wire Line
+	11150 5100 10600 5100
 Wire Wire Line
 	11950 5300 11850 5300
@@
 	1    0    0    -1
 $EndComp
-Text Label 11100 5100 0    60   ~ 0
+Text Label 10600 5100 0    60   ~ 0
 CAM_PHOTO
-Text Label 11100 5200 0    60   ~ 0
+Text Label 10600 5200 0    60   ~ 0
 CAM_PWR
-Text Label 11100 5000 0    60   ~ 0
+Text Label 10600 5000 0    60   ~ 0
 CAM_LED
 $Comp
 L R R10
 U 1 1 5A6750C6
-P 11800 5100
-F 0 "R10" V 11880 5100 50  0000 C CNN
-F 1 "4.7K" V 11800 5100 50  0000 C CNN
-F 2 "Resistors_SMD:R_0805" V 11730 5100 50  0001 C CNN
-F 3 "" H 11800 5100 50  0001 C CNN
-	1    11800 5100
+P 11300 5100
+F 0 "R10" V 11380 5100 50  0000 C CNN
+F 1 "4.7K" V 11300 5100 50  0000 C CNN
+F 2 "Resistors_SMD:R_0805" V 11230 5100 50  0001 C CNN
+F 3 "" H 11300 5100 50  0001 C CNN
+	1    11300 5100
 	0    1    1    0
 $EndComp
 Wire Wire Line
-	11950 5100 11950 5100
+	11450 5100 11950 5100
 Wire Wire Line
 	4800 5200 4200 5200
@@
 L R R9
 U 1 1 5A6780EF
-P 11800 5000
-F 0 "R9" V 11880 5000 50  0000 C CNN
-F 1 "0" V 11800 5000 50  0000 C CNN
-F 2 "Resistors_SMD:R_0805" V 11730 5000 50  0001 C CNN
-F 3 "" H 11800 5000 50  0001 C CNN
-	1    11800 5000
+P 11300 5000
+F 0 "R9" V 11380 5000 50  0000 C CNN
+F 1 "0" V 11300 5000 50  0000 C CNN
+F 2 "Resistors_SMD:R_0805" V 11230 5000 50  0001 C CNN
+F 3 "" H 11300 5000 50  0001 C CNN
+	1    11300 5000
 	0    1    1    0
 $EndComp
@@
 L R R11
 U 1 1 5A67821D
-P 11800 5200
-F 0 "R11" V 11880 5200 50  0000 C CNN
-F 1 "0" V 11800 5200 50  0000 C CNN
-F 2 "Resistors_SMD:R_0805" V 11730 5200 50  0001 C CNN
-F 3 "" H 11800 5200 50  0001 C CNN
-	1    11800 5200
+P 11300 5200
+F 0 "R11" V 11380 5200 50  0000 C CNN
+F 1 "0" V 11300 5200 50  0000 C CNN
+F 2 "Resistors_SMD:R_0805" V 11230 5200 50  0001 C CNN
+F 3 "" H 11300 5200 50  0001 C CNN
+	1    11300 5200
 	0    1    1    0
 $EndComp
@@
 P 8300 5450
 F 0 "R2" V 8380 5450 50  0000 C CNN
-F 1 "1k" V 8300 5450 50  0000 C CNN
+F 1 "2k7" V 8300 5450 50  0000 C CNN
 F 2 "Resistors_SMD:R_0805" V 8230 5450 50  0001 C CNN
 F 3 "" H 8300 5450 50  0001 C CNN
@@
 P 8300 5850
 F 0 "R3" V 8380 5850 50  0000 C CNN
-F 1 "1k" V 8300 5850 50  0000 C CNN
+F 1 "4k7" V 8300 5850 50  0000 C CNN
 F 2 "Resistors_SMD:R_0805" V 8230 5850 50  0001 C CNN
 F 3 "" H 8300 5850 50  0001 C CNN
@@
 $EndComp
 Connection ~ 14400 7450
+$Comp
+L R R38
+U 1 1 5A70F950
+P 11500 5450
+F 0 "R38" V 11580 5450 50  0000 C CNN
+F 1 "0" V 11500 5450 50  0000 C CNN
+F 2 "Resistors_SMD:R_0805" V 11430 5450 50  0001 C CNN
+F 3 "" H 11500 5450 50  0001 C CNN
+	1    11500 5450
+	-1   0    0    1
+$EndComp
+$Comp
+L R R39
+U 1 1 5A70FAC8
+P 11600 5450
+F 0 "R39" V 11680 5450 50  0000 C CNN
+F 1 "0" V 11600 5450 50  0000 C CNN
+F 2 "Resistors_SMD:R_0805" V 11530 5450 50  0001 C CNN
+F 3 "" H 11600 5450 50  0001 C CNN
+	1    11600 5450
+	-1   0    0    1
+$EndComp
+$Comp
+L R R40
+U 1 1 5A70FBEF
+P 11700 5450
+F 0 "R40" V 11780 5450 50  0000 C CNN
+F 1 "0" V 11700 5450 50  0000 C CNN
+F 2 "Resistors_SMD:R_0805" V 11630 5450 50  0001 C CNN
+F 3 "" H 11700 5450 50  0001 C CNN
+	1    11700 5450
+	-1   0    0    1
+$EndComp
+Wire Wire Line
+	11950 5200 11450 5200
+Wire Wire Line
+	11450 5000 11950 5000
+Wire Wire Line
+	11500 5300 11500 5200
+Connection ~ 11500 5200
+Wire Wire Line
+	11600 5300 11600 5100
+Connection ~ 11600 5100
+Wire Wire Line
+	11700 5300 11700 5000
+Connection ~ 11700 5000
+Wire Wire Line
+	11500 5600 11500 5750
+Wire Wire Line
+	11600 5600 11600 5850
+Wire Wire Line
+	11700 5750 11700 5600
+Wire Wire Line
+	11500 5750 11700 5750
+Connection ~ 11600 5750
+$Comp
+L GND #PWR036
+U 1 1 5A7112E1
+P 11600 5850
+F 0 "#PWR036" H 11600 5600 50  0001 C CNN
+F 1 "GND" H 11600 5700 50  0000 C CNN
+F 2 "" H 11600 5850 50  0001 C CNN
+F 3 "" H 11600 5850 50  0001 C CNN
+	1    11600 5850
+	1    0    0    -1
+$EndComp
 $EndSCHEMATC

Commit message: work review
Parts:
- added R41: 10k, Resistors_SMD:R_0805, symbol R
Connections:
- net +3V3: no longer U2.10 (OE)
- net GND: now also R41.1
- net OE: now reaches U1.54 ((A9)PC1)
- net OE: now also U2.10 (OE), R41.2
Changed lines of the file:
@@
 LIBS:TXB0104DR
 LIBS:LOGIC-TXS0108EPWR_TSSOP20_
-LIBS:CurrentControlSystems
 LIBS:Draco-cache
 EELAYER 25 0
@@
 $EndComp
 $Comp
-L GND #PWR01
+L GND #PWR14
 U 1 1 5A5AD6B5
 P 6350 7900
-F 0 "#PWR01" H 6350 7650 50  0001 C CNN
+F 0 "#PWR14" H 6350 7650 50  0001 C CNN
 F 1 "GND" H 6350 7750 50  0000 C CNN
 F 2 "" H 6350 7900 50  0001 C CNN
@@
 $EndComp
 $Comp
-L GND #PWR02
+L GND #PWR15
 U 1 1 5A5AD9C5
 P 6700 1850
-F 0 "#PWR02" H 6700 1600 50  0001 C CNN
+F 0 "#PWR15" H 6700 1600 50  0001 C CNN
 F 1 "GND" H 6700 1700 50  0000 C CNN
 F 2 "" H 6700 1850 50  0001 C CNN
@@
 $EndComp
 $Comp
-L +5V #PWR03
+L +5V #PWR12
 U 1 1 5A5ADA1C
 P 5750 1700
-F 0 "#PWR03" H 5750 1550 50  0001 C CNN
+F 0 "#PWR12" H 5750 1550 50  0001 C CNN
 F 1 "+5V" H 5750 1840 50  0000 C CNN
 F 2 "" H 5750 1700 50  0001 C CNN
@@
 $EndComp
 $Comp
-L +5V #PWR04
+L +5V #PWR13
 U 1 1 5A5ADA3E
 P 6250 1200
-F 0 "#PWR04" H 6250 1050 50  0001 C CNN
+F 0 "#PWR13" H 6250 1050 50  0001 C CNN
 F 1 "+5V" H 6250 1340 50  0000 C CNN
 F 2 "" H 6250 1200 50  0001 C CNN
@@
 $EndComp
 $Comp
-L GND #PWR05
+L GND #PWR6
 U 1 1 5A5ADF55
 P 3800 2850
-F 0 "#PWR05" H 3800 2600 50  0001 C CNN
+F 0 "#PWR6" H 3800 2600 50  0001 C CNN
 F 1 "GND" H 3800 2700 50  0000 C CNN
 F 2 "" H 3800 2850 50  0001 C CNN
@@
 $EndComp
 $Comp
-L +5V #PWR06
+L +5V #PWR9
 U 1 1 5A5AE55C
 P 4650 1700
-F 0 "#PWR06" H 4650 1550 50  0001 C CNN
+F 0 "#PWR9" H 4650 1550 50  0001 C CNN
 F 1 "+5V" H 4650 1840 50  0000 C CNN
 F 2 "" H 4650 1700 50  0001 C CNN
@@
 DTR
 $Comp
-L +5V #PWR07
+L +5V #PWR10
 U 1 1 5A5AEA3F
 P 4700 7400
-F 0 "#PWR07" H 4700 7250 50  0001 C CNN
+F 0 "#PWR10" H 4700 7250 50  0001 C CNN
 F 1 "+5V" H 4700 7540 50  0000 C CNN
 F 2 "" H 4700 7400 50  0001 C CNN
@@
 $EndComp
 $Comp
-L +5V #PWR08
+L +5V #PWR23
 U 1 1 5A5AF01F
 P 10250 8900
-F 0 "#PWR08" H 10250 8750 50  0001 C CNN
+F 0 "#PWR23" H 10250 8750 50  0001 C CNN
 F 1 "+5V" H 10250 9040 50  0000 C CNN
 F 2 "" H 10250 8900 50  0001 C CNN
@@
 $EndComp
 $Comp
-L GND #PWR09
+L GND #PWR24
 U 1 1 5A5AF162
 P 10250 9650
-F 0 "#PWR09" H 10250 9400 50  0001 C CNN
+F 0 "#PWR24" H 10250 9400 50  0001 C CNN
 F 1 "GND" H 10250 9500 50  0000 C CNN
 F 2 "" H 10250 9650 50  0001 C CNN
@@
 $EndComp
 $Comp
-L GND #PWR010
+L GND #PWR11
 U 1 1 5A5B0191
 P 4700 7800
-F 0 "#PWR010" H 4700 7550 50  0001 C CNN
+F 0 "#PWR11" H 4700 7550 50  0001 C CNN
 F 1 "GND" H 4700 7650 50  0000 C CNN
 F 2 "" H 4700 7800 50  0001 C CNN
@@
 $EndComp
 $Comp
-L GND #PWR011
+L GND #PWR8
 U 1 1 5A5B0AE7
 P 4050 9650
-F 0 "#PWR011" H 4050 9400 50  0001 C CNN
+F 0 "#PWR8" H 4050 9400 50  0001 C CNN
 F 1 "GND" H 4050 9500 50  0000 C CNN
 F 2 "" H 4050 9650 50  0001 C CNN
@@
 $EndComp
 $Comp
-L +5V #PWR012
+L +5V #PWR7
 U 1 1 5A5B0B22
 P 4050 8950
-F 0 "#PWR012" H 4050 8800 50  0001 C CNN
+F 0 "#PWR7" H 4050 8800 50  0001 C CNN
 F 1 "+5V" H 4050 9090 50  0000 C CNN
 F 2 "" H 4050 8950 50  0001 C CNN
@@
 PROG_RX
 $Comp
-L +5V #PWR013
+L +5V #PWR16
 U 1 1 5A5B171C
 P 8100 8800
-F 0 "#PWR013" H 8100 8650 50  0001 C CNN
+F 0 "#PWR16" H 8100 8650 50  0001 C CNN
 F 1 "+5V" H 8100 8940 50  0000 C CNN
 F 2 "" H 8100 8800 50  0001 C CNN
@@
 $EndComp
 $Comp
-L GND #PWR014
+L GND #PWR17
 U 1 1 5A5B32D0
 P 8100 9550
-F 0 "#PWR014" H 8100 9300 50  0001 C CNN
+F 0 "#PWR17" H 8100 9300 50  0001 C CNN
 F 1 "GND" H 8100 9400 50  0000 C CNN
 F 2 "" H 8100 9550 50  0001 C CNN
@@
 $EndComp
 $Comp
-L GND #PWR015
+L GND #PWR2
 U 1 1 5A5B6B40
 P 1700 8200
-F 0 "#PWR015" H 1700 7950 50  0001 C CNN
+F 0 "#PWR2" H 1700 7950 50  0001 C CNN
 F 1 "GND" H 1700 8050 50  0000 C CNN
 F 2 "" H 1700 8200 50  0001 C CNN
@@
 $EndComp
 $Comp
-L +3.3V #PWR016
+L +3.3V #PWR35
 U 1 1 5A5F2E73
 P 15150 6850
-F 0 "#PWR016" H 15150 6700 50  0001 C CNN
+F 0 "#PWR35" H 15150 6700 50  0001 C CNN
 F 1 "+3.3V" H 15150 6990 50  0000 C CNN
 F 2 "" H 15150 6850 50  0001 C CNN
@@
 $EndComp
 $Comp
-L GND #PWR017
+L GND #PWR36
 U 1 1 5A5F2FE9
 P 15150 8600
-F 0 "#PWR017" H 15150 8350 50  0001 C CNN
+F 0 "#PWR36" H 15150 8350 50  0001 C CNN
 F 1 "GND" H 15150 8450 50  0000 C CNN
 F 2 "" H 15150 8600 50  0001 C CNN
@@
 $EndComp
 $Comp
-L GND #PWR018
+L GND #PWR30
 U 1 1 5A60772E
 P 11950 8550
-F 0 "#PWR018" H 11950 8300 50  0001 C CNN
+F 0 "#PWR30" H 11950 8300 50  0001 C CNN
 F 1 "GND" H 11950 8400 50  0000 C CNN
 F 2 "" H 11950 8550 50  0001 C CNN
@@
 $EndComp
 $Comp
-L +5V #PWR019
+L +5V #PWR31
 U 1 1 5A6077D0
 P 12050 7200
-F 0 "#PWR019" H 12050 7050 50  0001 C CNN
+F 0 "#PWR31" H 12050 7050 50  0001 C CNN
 F 1 "+5V" H 12050 7340 50  0000 C CNN
 F 2 "" H 12050 7200 50  0001 C CNN
@@
 $EndComp
 $Comp
-L +3.3V #PWR020
+L +3.3V #PWR29
 U 1 1 5A607872
 P 11850 7200
-F 0 "#PWR020" H 11850 7050 50  0001 C CNN
+F 0 "#PWR29" H 11850 7050 50  0001 C CNN
 F 1 "+3.3V" H 11850 7340 50  0000 C CNN
 F 2 "" H 11850 7200 50  0001 C CNN
@@
 $EndComp
 $Comp
-L +3.3V #PWR021
+L +3.3V #PWR33
 U 1 1 5A60431F
 P 13700 4500
-F 0 "#PWR021" H 13700 4350 50  0001 C CNN
+F 0 "#PWR33" H 13700 4350 50  0001 C CNN
 F 1 "+3.3V" H 13700 4640 50  0000 C CNN
 F 2 "" H 13700 4500 50  0001 C CNN
@@
 $EndComp
 $Comp
-L GND #PWR022
+L GND #PWR34
 U 1 1 5A6046F8
 P 13700 5850
-F 0 "#PWR022" H 13700 5600 50  0001 C CNN
+F 0 "#PWR34" H 13700 5600 50  0001 C CNN
 F 1 "GND" H 13700 5700 50  0000 C CNN
 F 2 "" H 13700 5850 50  0001 C CNN
@@
 $EndComp
 $Comp
-L GND #PWR023
+L GND #PWR37
 U 1 1 5A641F11
 P 15750 7250
-F 0 "#PWR023" H 15750 7000 50  0001 C CNN
+F 0 "#PWR37" H 15750 7000 50  0001 C CNN
 F 1 "GND" H 15750 7100 50  0000 C CNN
 F 2 "" H 15750 7250 50  0001 C CNN
@@
 $EndComp
 $Comp
-L GND #PWR024
+L GND #PWR32
 U 1 1 5A662ADC
 P 13350 5850
-F 0 "#PWR024" H 13350 5600 50  0001 C CNN
+F 0 "#PWR32" H 13350 5600 50  0001 C CNN
 F 1 "GND" H 13350 5700 50  0000 C CNN
 F 2 "" H 13350 5850 50  0001 C CNN
@@
 $EndComp
 $Comp
-L +5V #PWR025
+L +5V #PWR3
 U 1 1 5A66CBF6
 P 2250 2550
-F 0 "#PWR025" H 2250 2400 50  0001 C CNN
+F 0 "#PWR3" H 2250 2400 50  0001 C CNN
 F 1 "+5V" H 2250 2690 50  0000 C CNN
 F 2 "" H 2250 2550 50  0001 C CNN
@@
 	11950 8500 11950 8550
 Wire Wire Line
-	11400 7250 11850 7250
-Connection ~ 11850 7250
-Wire Wire Line
 	12400 7600 13100 7600
 Wire Wire Line
@@
 	11500 7500 11400 7500
 Wire Wire Line
-	11400 7500 11400 7250
+	11400 7250 11400 7500
 Wire Wire Line
 	15700 7600 16200 7600
@@
 	11850 5300 11850 5400
 $Comp
-L GND #PWR026
+L GND #PWR28
 U 1 1 5A672143
 P 11850 5400
-F 0 "#PWR026" H 11850 5150 50  0001 C CNN
+F 0 "#PWR28" H 11850 5150 50  0001 C CNN
 F 1 "GND" H 11850 5250 50  0000 C CNN
 F 2 "" H 11850 5400 50  0001 C CNN
@@
 $EndComp
 $Comp
-L GND #PWR027
+L GND #PWR25
 U 1 1 5A67CAA7
 P 10300 5250
-F 0 "#PWR027" H 10300 5000 50  0001 C CNN
+F 0 "#PWR25" H 10300 5000 50  0001 C CNN
 F 1 "GND" H 10300 5100 50  0000 C CNN
 F 2 "" H 10300 5250 50  0001 C CNN
@@
 $EndComp
 $Comp
-L GND #PWR028
+L GND #PWR22
 U 1 1 5A67CBBA
 P 9900 5250
-F 0 "#PWR028" H 9900 5000 50  0001 C CNN
+F 0 "#PWR22" H 9900 5000 50  0001 C CNN
 F 1 "GND" H 9900 5100 50  0000 C CNN
 F 2 "" H 9900 5250 50  0001 C CNN
@@
 $EndComp
 $Comp
-L GND #PWR029
+L GND #PWR19
 U 1 1 5A67CCCD
 P 9500 5250
-F 0 "#PWR029" H 9500 5000 50  0001 C CNN
+F 0 "#PWR19" H 9500 5000 50  0001 C CNN
 F 1 "GND" H 9500 5100 50  0000 C CNN
 F 2 "" H 9500 5250 50  0001 C CNN
@@
 $EndComp
 $Comp
-L GND #PWR030
+L GND #PWR21
 U 1 1 5A68BFAE
 P 9800 7950
-F 0 "#PWR030" H 9800 7700 50  0001 C CNN
+F 0 "#PWR21" H 9800 7700 50  0001 C CNN
 F 1 "GND" H 9800 7800 50  0000 C CNN
 F 2 "" H 9800 7950 50  0001 C CNN
@@
 $EndComp
 $Comp
-L +BATT #PWR031
+L +BATT #PWR20
 U 1 1 5A68C099
 P 9800 7100
-F 0 "#PWR031" H 9800 6950 50  0001 C CNN
+F 0 "#PWR20" H 9800 6950 50  0001 C CNN
 F 1 "+BATT" H 9800 7240 50  0000 C CNN
 F 2 "" H 9800 7100 50  0001 C CNN
@@
 $EndComp
 $Comp
-L GND #PWR032
+L GND #PWR18
 U 1 1 5A6DAD78
 P 8300 6050
-F 0 "#PWR032" H 8300 5800 50  0001 C CNN
+F 0 "#PWR18" H 8300 5800 50  0001 C CNN
 F 1 "GND" H 8300 5900 50  0000 C CNN
 F 2 "" H 8300 6050 50  0001 C CNN
@@
 	3550 4800 3550 4900
 $Comp
-L GND #PWR033
+L GND #PWR5
 U 1 1 5A6A2B9C
 P 3550 4900
-F 0 "#PWR033" H 3550 4650 50  0001 C CNN
+F 0 "#PWR5" H 3550 4650 50  0001 C CNN
 F 1 "GND" H 3550 4750 50  0000 C CNN
 F 2 "" H 3550 4900 50  0001 C CNN
@@
 $EndComp
 $Comp
-L +5V #PWR034
+L +5V #PWR4
 U 1 1 5A6A2F82
 P 3550 4400
-F 0 "#PWR034" H 3550 4250 50  0001 C CNN
+F 0 "#PWR4" H 3550 4250 50  0001 C CNN
 F 1 "+5V" H 3550 4540 50  0000 C CNN
 F 2 "" H 3550 4400 50  0001 C CNN
@@
 $EndComp
 $Comp
-L +BATT #PWR035
+L +BATT #PWR1
 U 1 1 5A6A6502
 P 1450 2550
-F 0 "#PWR035" H 1450 2400 50  0001 C CNN
+F 0 "#PWR1" H 1450 2400 50  0001 C CNN
 F 1 "+BATT" H 1450 2690 50  0000 C CNN
 F 2 "" H 1450 2550 50  0001 C CNN
@@
 $EndComp
 Wire Wire Line
-	11950 5200 11450 5200
+	11450 5200 11950 5200
 Wire Wire Line
 	11450 5000 11950 5000
@@
 Connection ~ 11600 5750
 $Comp
-L GND #PWR036
+L GND #PWR27
 U 1 1 5A7112E1
 P 11600 5850
-F 0 "#PWR036" H 11600 5600 50  0001 C CNN
+F 0 "#PWR27" H 11600 5600 50  0001 C CNN
 F 1 "GND" H 11600 5700 50  0000 C CNN
 F 2 "" H 11600 5850 50  0001 C CNN
@@
 	1    0    0    -1
 $EndComp
+Wire Wire Line
+	10150 7250 11400 7250
+Text Label 10150 7250 0    60   ~ 0
+OE
+$Comp
+L R R41
+U 1 1 5A700696
+P 10550 7500
+F 0 "R41" V 10630 7500 50  0000 C CNN
+F 1 "10k" V 10550 7500 50  0000 C CNN
+F 2 "Resistors_SMD:R_0805" V 10480 7500 50  0001 C CNN
+F 3 "" H 10550 7500 50  0001 C CNN
+	1    10550 7500
+	-1   0    0    1
+$EndComp
+$Comp
+L GND #PWR26
+U 1 1 5A7007E7
+P 10550 7700
+F 0 "#PWR26" H 10550 7450 50  0001 C CNN
+F 1 "GND" H 10550 7550 50  0000 C CNN
+F 2 "" H 10550 7700 50  0001 C CNN
+F 3 "" H 10550 7700 50  0001 C CNN
+	1    10550 7700
+	1    0    0    -1
+$EndComp
+Wire Wire Line
+	10550 7700 10550 7650
+Wire Wire Line
+	10550 7350 10550 7250
+Connection ~ 10550 7250
+Wire Wire Line
+	7400 4100 8050 4100
+Text Label 8050 4100 2    60   ~ 0
+OE
 $EndSCHEMATC
