File: gps.sch (KiCad schematic (older format))
At the start: 4 parts, among them U5 SAM-M8Q

Commit message: Did design review. Changed/confirmed voltage levels
Parts:
- BT1: footprint (none) -> Battery_Holders:Keystone_3000_1x12mm-CoinCell
- C25: renamed from C23; footprint (none) -> Capacitors_SMD:C_0805
- C26: renamed from C24; footprint (none) -> Capacitors_SMD:C_0805
- renumbered U5 to U6
Connections:
- net +5V is gone; now on net +3V3: C25.1, U6.2 (VCC_IO)
- net GPS_INT: now reaches U6.19 (EXTINT)
Changed lines of the file:
@@
 $EndDescr
 $Comp
-L SAM-M8Q U5
+L SAM-M8Q U6
 U 1 1 5A5DC8DE
 P 5700 3950
-F 0 "U5" H 5100 4600 60  0000 L CNN
+F 0 "U6" H 5100 4600 60  0000 L CNN
 F 1 "SAM-M8Q" H 5100 4500 60  0000 L CNN
 F 2 "" H 5700 3950 60  0001 C CNN
@@
 $EndComp
 $Comp
-L GND #PWR047
+L GND #PWR058
 U 1 1 5A5DC941
 P 5700 4600
-F 0 "#PWR047" H 5700 4350 50  0001 C CNN
+F 0 "#PWR058" H 5700 4350 50  0001 C CNN
 F 1 "GND" H 5700 4450 50  0000 C CNN
 F 2 "" H 5700 4600 50  0001 C CNN
@@
 $EndComp
 $Comp
-L +5V #PWR048
-U 1 1 5A5DC973
-P 3500 3450
-F 0 "#PWR048" H 3500 3300 50  0001 C CNN
-F 1 "+5V" H 3500 3590 50  0000 C CNN
-F 2 "" H 3500 3450 50  0001 C CNN
-F 3 "" H 3500 3450 50  0001 C CNN
-	1    3500 3450
-	1    0    0    -1
-$EndComp
-$Comp
-L +3.3V #PWR049
+L +3.3V #PWR059
 U 1 1 5A5DC989
 P 3800 3450
-F 0 "#PWR049" H 3800 3300 50  0001 C CNN
+F 0 "#PWR059" H 3800 3300 50  0001 C CNN
 F 1 "+3.3V" H 3800 3590 50  0000 C CNN
 F 2 "" H 3800 3450 50  0001 C CNN
@@
 F 0 "BT1" H 4900 4700 50  0000 L CNN
 F 1 "Battery_Cell" H 4900 4600 50  0000 L CNN
-F 2 "" V 4800 4660 50  0001 C CNN
+F 2 "Battery_Holders:Keystone_3000_1x12mm-CoinCell" V 4800 4660 50  0001 C CNN
 F 3 "" V 4800 4660 50  0001 C CNN
 	1    4800 4600
@@
 $EndComp
 $Comp
-L GND #PWR050
+L GND #PWR060
 U 1 1 5A5DCA28
 P 4800 4750
-F 0 "#PWR050" H 4800 4500 50  0001 C CNN
+F 0 "#PWR060" H 4800 4500 50  0001 C CNN
 F 1 "GND" H 4800 4600 50  0000 C CNN
 F 2 "" H 4800 4750 50  0001 C CNN
@@
 GPS_SDA
 $Comp
-L C C23
+L C C25
 U 1 1 5A5DDFEA
 P 3500 4050
-F 0 "C23" H 3525 4150 50  0000 L CNN
+F 0 "C25" H 3525 4150 50  0000 L CNN
 F 1 "100nF" H 3525 3950 50  0000 L CNN
-F 2 "" H 3538 3900 50  0001 C CNN
+F 2 "Capacitors_SMD:C_0805" H 3538 3900 50  0001 C CNN
 F 3 "" H 3500 4050 50  0001 C CNN
 	1    3500 4050
@@
 $EndComp
 $Comp
-L C C24
+L C C26
 U 1 1 5A5DE04A
 P 3800 4050
-F 0 "C24" H 3825 4150 50  0000 L CNN
+F 0 "C26" H 3825 4150 50  0000 L CNN
 F 1 "100nF" H 3825 3950 50  0000 L CNN
-F 2 "" H 3838 3900 50  0001 C CNN
+F 2 "Capacitors_SMD:C_0805" H 3838 3900 50  0001 C CNN
 F 3 "" H 3800 4050 50  0001 C CNN
 	1    3800 4050
@@
 $EndComp
 $Comp
-L GND #PWR051
+L GND #PWR061
 U 1 1 5A5DE074
 P 3500 4350
-F 0 "#PWR051" H 3500 4100 50  0001 C CNN
+F 0 "#PWR061" H 3500 4100 50  0001 C CNN
 F 1 "GND" H 3500 4200 50  0000 C CNN
 F 2 "" H 3500 4350 50  0001 C CNN
@@
 Wire Wire Line
 	5700 4550 5700 4600
+Wire Wire Line
+	6500 3850 6800 3850
+Text HLabel 6800 3850 2    60   Output ~ 0
+GPS_INT
+$Comp
+L +3.3V #PWR062
+U 1 1 5A6D5EDC
+P 3500 3450
+F 0 "#PWR062" H 3500 3300 50  0001 C CNN
+F 1 "+3.3V" H 3500 3590 50  0000 C CNN
+F 2 "" H 3500 3450 50  0001 C CNN
+F 3 "" H 3500 3450 50  0001 C CNN
+	1    3500 3450
+	1    0    0    -1
+$EndComp
 $EndSCHEMATC

Commit message: Started Board layout
Parts:
- U6: footprint (none) -> Current_Control_Systems:SAM-M8Q
Changed lines of the file:
@@
 LIBS:TXB0104DR
 LIBS:LOGIC-TXS0108EPWR_TSSOP20_
+LIBS:CurrentControlSystems
 LIBS:Draco-cache
 EELAYER 25 0
@@
 F 0 "U6" H 5100 4600 60  0000 L CNN
 F 1 "SAM-M8Q" H 5100 4500 60  0000 L CNN
-F 2 "" H 5700 3950 60  0001 C CNN
+F 2 "Current_Control_Systems:SAM-M8Q" H 5700 3950 60  0001 C CNN
 F 3 "" H 5700 3950 60  0001 C CNN
 	1    5700 3950
@@
 $EndComp
 $Comp
-L GND #PWR058
+L GND #PWR059
 U 1 1 5A5DC941
 P 5700 4600
-F 0 "#PWR058" H 5700 4350 50  0001 C CNN
+F 0 "#PWR059" H 5700 4350 50  0001 C CNN
 F 1 "GND" H 5700 4450 50  0000 C CNN
 F 2 "" H 5700 4600 50  0001 C CNN
@@
 $EndComp
 $Comp
-L +3.3V #PWR059
+L +3.3V #PWR060
 U 1 1 5A5DC989
 P 3800 3450
-F 0 "#PWR059" H 3800 3300 50  0001 C CNN
+F 0 "#PWR060" H 3800 3300 50  0001 C CNN
 F 1 "+3.3V" H 3800 3590 50  0000 C CNN
 F 2 "" H 3800 3450 50  0001 C CNN
@@
 $EndComp
 $Comp
-L GND #PWR060
+L GND #PWR061
 U 1 1 5A5DCA28
 P 4800 4750
-F 0 "#PWR060" H 4800 4500 50  0001 C CNN
+F 0 "#PWR061" H 4800 4500 50  0001 C CNN
 F 1 "GND" H 4800 4600 50  0000 C CNN
 F 2 "" H 4800 4750 50  0001 C CNN
@@
 $EndComp
 $Comp
-L GND #PWR061
+L GND #PWR062
 U 1 1 5A5DE074
 P 3500 4350
-F 0 "#PWR061" H 3500 4100 50  0001 C CNN
+F 0 "#PWR062" H 3500 4100 50  0001 C CNN
 F 1 "GND" H 3500 4200 50  0000 C CNN
 F 2 "" H 3500 4350 50  0001 C CNN
@@
 GPS_INT
 $Comp
-L +3.3V #PWR062
+L +3.3V #PWR063
 U 1 1 5A6D5EDC
 P 3500 3450
-F 0 "#PWR062" H 3500 3300 50  0001 C CNN
+F 0 "#PWR063" H 3500 3300 50  0001 C CNN
 F 1 "+3.3V" H 3500 3590 50  0000 C CNN
 F 2 "" H 3500 3450 50  0001 C CNN
