File: launch.sch (KiCad schematic (older format))
At the start: 24 parts, among them J17 CHARGE_A, J18 CHARGE_C, J19 CHARGE_B, Q1 BC817, Q2 Q_NMOS_DGS, Q3 BC817, Q4 Q_NMOS_DGS, Q5 BC817, Q6 Q_NMOS_DGS

Commit message: Fixed MOSFET pinout
Parts:
- removed Q2, Q4, Q6: Q_NMOS_DGS, TO_SOT_Packages_SMD:TO-252-2, symbol Q_NMOS_DGS
- added Q2, Q4, Q6: Q_NMOS_GDS, TO_SOT_Packages_SMD:TO-252-2, symbol Q_NMOS_GDS
Connections:
- net GND: now also Q2.3 (S), Q4.3 (S), Q6.3 (S)
- net at J17.2 (Pin_2), R13.1: now also Q2.2 (D)
- net at R15.2: now also Q2.1 (G)
- net at J19.2 (Pin_2), R22.1: now also Q6.2 (D)
- net at R25.2: now also Q6.1 (G)
- net at J18.2 (Pin_2), R18.1: now also Q4.2 (D)
- net at R21.2: now also Q4.1 (G)
Changed lines of the file:
@@
 LIBS:TXB0104DR
 LIBS:LOGIC-TXS0108EPWR_TSSOP20_
-LIBS:CurrentControlSystems
 LIBS:Draco-cache
 EELAYER 25 0
@@
 Text HLabel 1950 2400 0    60   Output ~ 0
 TEST_READ_A
-$Comp
-L Q_NMOS_DGS Q2
-U 1 1 5A5BF6EC
-P 3600 3050
-F 0 "Q2" H 3800 3100 50  0000 L CNN
-F 1 "Q_NMOS_DGS" H 3800 3000 50  0000 L CNN
-F 2 "TO_SOT_Packages_SMD:TO-252-2" H 3800 3150 50  0001 C CNN
-F 3 "" H 3600 3050 50  0001 C CNN
-	1    3600 3050
-	-1   0    0    -1
-$EndComp
 Wire Wire Line
 	3500 3250 3500 3500
@@
 Text HLabel 6750 2400 0    60   Output ~ 0
 TEST_READ_B
-$Comp
-L Q_NMOS_DGS Q6
-U 1 1 5A5C03EB
-P 8400 3050
-F 0 "Q6" H 8600 3100 50  0000 L CNN
-F 1 "Q_NMOS_DGS" H 8600 3000 50  0000 L CNN
-F 2 "TO_SOT_Packages_SMD:TO-252-2" H 8600 3150 50  0001 C CNN
-F 3 "" H 8400 3050 50  0001 C CNN
-	1    8400 3050
-	-1   0    0    -1
-$EndComp
 Wire Wire Line
 	8300 3250 8300 3500
@@
 Text HLabel 4700 4750 0    60   Output ~ 0
 TEST_READ_C
-$Comp
-L Q_NMOS_DGS Q4
-U 1 1 5A5C9B20
-P 6350 5400
-F 0 "Q4" H 6550 5450 50  0000 L CNN
-F 1 "Q_NMOS_DGS" H 6550 5350 50  0000 L CNN
-F 2 "TO_SOT_Packages_SMD:TO-252-2" H 6550 5500 50  0001 C CNN
-F 3 "" H 6350 5400 50  0001 C CNN
-	1    6350 5400
-	-1   0    0    -1
-$EndComp
 Wire Wire Line
 	6250 5600 6250 5850
@@
 	1    0    0    -1
 $EndComp
+$Comp
+L Q_NMOS_GDS Q2
+U 1 1 5A72C2BC
+P 3600 3050
+F 0 "Q2" H 3800 3100 50  0000 L CNN
+F 1 "Q_NMOS_GDS" H 3800 3000 50  0000 L CNN
+F 2 "TO_SOT_Packages_SMD:TO-252-2" H 3800 3150 50  0001 C CNN
+F 3 "" H 3600 3050 50  0001 C CNN
+	1    3600 3050
+	-1   0    0    -1
+$EndComp
+$Comp
+L Q_NMOS_GDS Q6
+U 1 1 5A72C8F7
+P 8400 3050
+F 0 "Q6" H 8600 3100 50  0000 L CNN
+F 1 "Q_NMOS_GDS" H 8600 3000 50  0000 L CNN
+F 2 "TO_SOT_Packages_SMD:TO-252-2" H 8600 3150 50  0001 C CNN
+F 3 "" H 8400 3050 50  0001 C CNN
+	1    8400 3050
+	-1   0    0    -1
+$EndComp
+$Comp
+L Q_NMOS_GDS Q4
+U 1 1 5A72C98E
+P 6350 5400
+F 0 "Q4" H 6550 5450 50  0000 L CNN
+F 1 "Q_NMOS_GDS" H 6550 5350 50  0000 L CNN
+F 2 "TO_SOT_Packages_SMD:TO-252-2" H 6550 5500 50  0001 C CNN
+F 3 "" H 6350 5400 50  0001 C CNN
+	1    6350 5400
+	-1   0    0    -1
+$EndComp
 $EndSCHEMATC
